Commit message: right and left sides complete (no legs)

File: urdf_model/cricket_robot.urdf (robot description, URDF)
Before this commit: robot materials, 3 links, 1 joints
Links:
- removed link link_name
- added link left_box; visual box size=0.4 0.15 0.15
- added link left_cylinder; visual cylinder length=0.4 radius=0.075
- added link right_cylinder; visual cylinder length=0.4 radius=0.075
- link right_box: geometry visual box size=0.4 0.15 0.15
Joints:
- added joint body_to_left_box: type fixed, parent main_body, child left_box, origin xyz=0.0 -0.2 0.0
- added joint left_box-cylinder: type fixed, parent left_box, child left_cylinder
- added joint right_box-cylinder: type fixed, parent right_box, child right_cylinder

Commit message: main body complete and working

File: urdf_model/cricket_robot.urdf (robot description, URDF)
Before this commit: robot materials, 5 links, 4 joints
Links:
- removed link main_body
- added link base_link; visual box size=0.41 0.36 0.06
- link left_box: geometry visual box size=0.1 0.07 0.06
- link left_cylinder: geometry visual cylinder length=0.1 radius=0.03
- link right_box: geometry visual box size=0.1 0.07 0.06
- link right_cylinder: geometry visual cylinder length=0.1 radius=0.03
Joints:
- removed joint body_to_right_box
- added joint base_to_right_box: type fixed, parent base_link, child right_box
- joint body_to_left_box: origin xyz=0.0 -0.2 0.0 -> xyz=0.0 -0.18 0.0; parent main_body -> base_link

Commit message: shoulder right front

File: urdf_model/cricket_robot.urdf (robot description, URDF)
Before this commit: robot origins, 5 links, 4 joints
Links:
- added link frl_shoulder_cylinder; visual cylinder length=0.1 radius=0.03
Joints:
- added joint joint_name: type fixed, parent right_cylinder, child frl_shoulder_cylinder, origin xyz=0.5 0.25 0.0 rpy=0 0 0.0

Commit message: 4 shoulders completed

File: urdf_model/cricket_robot.urdf (robot description, URDF)
Before this commit: robot origins, 6 links, 5 joints
Links:
- added link bll_shoulder_box; visual box size=0.06 0.03 0.12
- added link bll_shoulder_cylinder; visual cylinder length=0.12 radius=0.03
- added link brl_shoulder_box; visual box size=0.06 0.03 0.12
- added link brl_shoulder_cylinder; visual cylinder length=0.12 radius=0.03
- added link fll_shoulder_box; visual box size=0.06 0.03 0.12
- added link fll_shoulder_cylinder; visual cylinder length=0.12 radius=0.03
- added link frl_shoulder_box; visual box size=0.06 0.03 0.12
- link frl_shoulder_cylinder: geometry visual cylinder length=0.12 radius=0.03
Joints:
- removed joint joint_name
- added joint bll_shoulder-body: type fixed, parent left_cylinder, child bll_shoulder_cylinder, origin xyz=-0.12 0.0 0.0 rpy=0 0 0.0
- added joint bll_shoulder_cyl-box: type fixed, parent bll_shoulder_cylinder, child bll_shoulder_box, origin xyz=0.0 -0.017 0.0 rpy=0.0 0.0 0.0
- added joint brl_shoulder-body: type fixed, parent right_cylinder, child brl_shoulder_cylinder, origin xyz=-0.12 0.0 0.0 rpy=0 0 0.0
- added joint brl_shoulder_cyl-box: type fixed, parent brl_shoulder_cylinder, child brl_shoulder_box, origin xyz=0.0 0.017 0.0 rpy=0.0 0.0 0.0
- added joint fll_shoulder-body: type fixed, parent left_cylinder, child fll_shoulder_cylinder, origin xyz=0.12 0.0 0.0 rpy=0 0 0.0
- added joint fll_shoulder_cyl-box: type fixed, parent fll_shoulder_cylinder, child fll_shoulder_box, origin xyz=0.0 -0.017 0.0 rpy=0.0 0.0 0.0
- added joint frl_shoulder-body: type fixed, parent right_cylinder, child frl_shoulder_cylinder, origin xyz=0.12 0.0 0.0 rpy=0 0 0.0
- added joint frl_shoulder_cyl-box: type fixed, parent frl_shoulder_cylinder, child frl_shoulder_box, origin xyz=0.0 0.017 0.0 rpy=0.0 0.0 0.0
- joint base_to_right_box: origin (none) -> xyz=0 0.215 0.0
- joint body_to_left_box: origin xyz=0.0 -0.18 0.0 -> xyz=0.0 -0.215 0.0
- joint left_box-cylinder: origin (none) -> xyz=0.0 -0.035 0.0
- joint right_box-cylinder: origin (none) -> xyz=0.0 0.035 0.0 rpy=0.0 0.0 0.0

Commit message: front right leg completed

File: urdf_model/cricket_robot.urdf (robot description, URDF)
Before this commit: robot origins, 13 links, 12 joints
Links:
- added link frl_ends_track; visual cylinder length=0.05 radius=0.03
- added link frl_jointed_track; visual cylinder length=0.05 radius=0.03
- added link frl_knee_base; visual box size=0.12 0.01 0.06
- added link frl_knee_box; visual box size=0.08 0.05 0.06
- added link frl_shoulder2_base; visual box size=0.05 0.01 0.06
- added link frl_shoulder2_box; visual box size=0.11 0.05 0.06
- added link frl_track; visual box size=0.190 0.05 0.06
- link frl_shoulder_box: geometry visual box size=0.12 0.03 0.06
- link left_box: geometry visual box size=0.1 0.04 0.06
- link right_box: geometry visual box size=0.1 0.04 0.06
Joints:
- added joint frl_ankle: type fixed, parent frl_knee_box, child frl_jointed_track, origin xyz=0.0 0.032 0.0 rpy=0.0 0.0 0.0
- added joint frl_final_track_joint: type fixed, parent frl_track, child frl_ends_track, origin xyz=0.095 0.0 0.0 rpy=0.0 0.0 0.0
- added joint frl_jointed_track-track: type fixed, parent frl_jointed_track, child frl_track, origin xyz=0.095 0.0 0.0 rpy=0.0 0.0 0.0
- added joint frl_knee_base-box: type fixed, parent frl_knee_base, child frl_knee_box, origin xyz=0.18 0.0 0.0 rpy=0.0 0.0 0.0
- added joint frl_shoulder2-knee: type fixed, parent frl_shoulder2_box, child frl_knee_base, origin xyz=0.0 0.052 0.0 rpy=0.0 0.0 0.0
- added joint frl_shoulder2-shoulder: type fixed, parent frl_shoulder_box, child frl_shoulder2_base, origin xyz=0.0 0.02 0.0 rpy=0.0 0.0 0.0
- added joint frl_shoulder2_base-box: type fixed, parent frl_shoulder2_base, child frl_shoulder2_box, origin xyz=-0.14 0.0 0.0 rpy=0.0 0.0 0.0
- joint base_to_right_box: origin xyz=0 0.215 0.0 -> xyz=0 0.2 0.0
- joint body_to_left_box: origin xyz=0.0 -0.215 0.0 -> xyz=0.0 -0.2 0.0
- joint frl_shoulder_cyl-box: origin xyz=0.0 0.017 0.0 rpy=0.0 0.0 0.0 -> xyz=0.05 0.017 0.0 rpy=0.0 0.0 0.0
- joint left_box-cylinder: origin xyz=0.0 -0.035 0.0 -> xyz=0.0 -0.02 0.0
- joint right_box-cylinder: origin xyz=0.0 0.035 0.0 rpy=0.0 0.0 0.0 -> xyz=0.0 0.02 0.0 rpy=0.0 0.0 0.0

Commit message: front legs completed

File: urdf_model/cricket_robot.urdf (robot description, URDF)
Before this commit: robot origins, 20 links, 19 joints
Links:
- added link fll_ends_track; visual cylinder length=0.05 radius=0.03
- added link fll_jointed_track; visual cylinder length=0.05 radius=0.03
- added link fll_knee_base; visual box size=0.12 0.01 0.06
- added link fll_knee_box; visual box size=0.08 0.05 0.06
- added link fll_shoulder2_base; visual box size=0.05 0.01 0.06
- added link fll_shoulder2_box; visual box size=0.11 0.05 0.06
- added link fll_track; visual box size=0.190 0.05 0.06
- link fll_shoulder_box: geometry visual box size=0.12 0.03 0.06
Joints:
- added joint fll_ankle: type fixed, parent fll_knee_box, child fll_jointed_track, origin xyz=0.0 -0.032 0.0 rpy=0.0 0.0 0.0
- added joint fll_final_track_joint: type fixed, parent fll_track, child fll_ends_track, origin xyz=0.095 0.0 0.0 rpy=0.0 0.0 0.0
- added joint fll_jointed_track-track: type fixed, parent fll_jointed_track, child fll_track, origin xyz=0.095 0.0 0.0 rpy=0.0 0.0 0.0
- added joint fll_knee_base-box: type fixed, parent fll_knee_base, child fll_knee_box, origin xyz=0.18 0.0 0.0 rpy=0.0 0.0 0.0
- added joint fll_shoulder2-knee: type fixed, parent fll_shoulder2_box, child fll_knee_base, origin xyz=0.0 -0.052 0.0 rpy=0.0 0.0 0.0
- added joint fll_shoulder2-shoulder: type fixed, parent fll_shoulder_box, child fll_shoulder2_base, origin xyz=0.0 -0.02 0.0 rpy=0.0 0.0 0.0
- added joint fll_shoulder2_base-box: type fixed, parent fll_shoulder2_base, child fll_shoulder2_box, origin xyz=-0.14 0.0 0.0 rpy=0.0 0.0 0.0
- joint fll_shoulder_cyl-box: origin xyz=0.0 -0.017 0.0 rpy=0.0 0.0 0.0 -> xyz=0.05 -0.017 0.0 rpy=0.0 0.0 0.0

Commit message: model completed

File: urdf_model/cricket_robot.urdf (robot description, URDF)
Before this commit: robot origins, 27 links, 26 joints
Links:
- added link bll_ends_track; visual cylinder length=0.05 radius=0.03
- added link bll_jointed_track; visual cylinder length=0.05 radius=0.03
- added link bll_knee_base; visual box size=0.12 0.01 0.06
- added link bll_knee_box; visual box size=0.08 0.05 0.06
- added link bll_shoulder2_base; visual box size=0.05 0.01 0.06
- added link bll_shoulder2_box; visual box size=0.11 0.05 0.06
- added link bll_track; visual box size=0.190 0.05 0.06
- added link brl_ends_track; visual cylinder length=0.05 radius=0.03
- added link brl_jointed_track; visual cylinder length=0.05 radius=0.03
- added link brl_knee_base; visual box size=0.12 0.01 0.06
- added link brl_knee_box; visual box size=0.08 0.05 0.06
- added link brl_shoulder2_base; visual box size=0.05 0.01 0.06
- added link brl_shoulder2_box; visual box size=0.11 0.05 0.06
- added link brl_track; visual box size=0.190 0.05 0.06
- link bll_shoulder_box: geometry visual box size=0.12 0.03 0.06
- link brl_shoulder_box: geometry visual box size=0.12 0.03 0.06
Joints:
- added joint bll_ankle: type fixed, parent bll_knee_box, child bll_jointed_track, origin xyz=0.0 -0.032 0.0 rpy=0.0 0.0 0.0
- added joint bll_final_track_joint: type fixed, parent bll_track, child bll_ends_track, origin xyz=-0.095 0.0 0.0 rpy=0.0 0.0 0.0
- added joint bll_jointed_track-track: type fixed, parent bll_jointed_track, child bll_track, origin xyz=0.095 0.0 0.0 rpy=0.0 3.14150 0.0
- added joint bll_knee_base-box: type fixed, parent bll_knee_base, child bll_knee_box, origin xyz=-0.18 0.0 0.0 rpy=0.0 0.0 0.0
- added joint bll_shoulder2-knee: type fixed, parent bll_shoulder2_box, child bll_knee_base, origin xyz=0.0 -0.052 0.0 rpy=0.0 0.0 0.0
- added joint bll_shoulder2-shoulder: type fixed, parent bll_shoulder_box, child bll_shoulder2_base, origin xyz=0.0 -0.02 0.0 rpy=0.0 0.0 0.0
- added joint bll_shoulder2_base-box: type fixed, parent bll_shoulder2_base, child bll_shoulder2_box, origin xyz=0.14 0.0 0.0 rpy=0.0 0.0 0.0
- added joint brl_ankle: type fixed, parent brl_knee_box, child brl_jointed_track, origin xyz=0.0 0.032 0.0 rpy=0.0 0.0 0.0
- added joint brl_final_track_joint: type fixed, parent brl_track, child brl_ends_track, origin xyz=-0.095 0.0 0.0 rpy=0.0 0.0 0.0
- added joint brl_jointed_track-track: type fixed, parent brl_jointed_track, child brl_track, origin xyz=0.095 0.0 0.0 rpy=0.0 3.14150 0.0
- added joint brl_knee_base-box: type fixed, parent brl_knee_base, child brl_knee_box, origin xyz=-0.18 0.0 0.0 rpy=0.0 0.0 0.0
- added joint brl_shoulder2-knee: type fixed, parent brl_shoulder2_box, child brl_knee_base, origin xyz=0.0 0.052 0.0 rpy=0.0 0.0 0.0
- added joint brl_shoulder2-shoulder: type fixed, parent brl_shoulder_box, child brl_shoulder2_base, origin xyz=0.0 0.02 0.0 rpy=0.0 0.0 0.0
- added joint brl_shoulder2_base-box: type fixed, parent brl_shoulder2_base, child brl_shoulder2_box, origin xyz=0.14 0.0 0.0 rpy=0.0 0.0 0.0
- joint bll_shoulder_cyl-box: origin xyz=0.0 -0.017 0.0 rpy=0.0 0.0 0.0 -> xyz=-0.05 -0.017 0.0 rpy=0.0 0.0 0.0
- joint brl_shoulder_cyl-box: origin xyz=0.0 0.017 0.0 rpy=0.0 0.0 0.0 -> xyz=-0.05 0.017 0.0 rpy=0.0 0.0 0.0

Commit message: movement and refactoring added

File: urdf_model/cricket_robot.urdf (robot description, URDF)
Before this commit: robot origins, 41 links, 40 joints
Joints:
- joint bll_ankle: axis (none) -> 0.0 1 0.0; type fixed -> continuous
- joint bll_final_track_joint: axis (none) -> 0.0 1 0.0; type fixed -> continuous
- joint bll_shoulder-body: axis (none) -> 1 0.0 0.0; limit (none) -> lower=-1.57075 upper=1.57075 effort=1000.0 velocity=0.5; type fixed -> revolute
- joint bll_shoulder2-knee: axis (none) -> 0.0 1 0.0; type fixed -> continuous
- joint bll_shoulder2-shoulder: axis (none) -> 0.0 1 0.0; type fixed -> continuous
- joint brl_ankle: axis (none) -> 0.0 1 0.0; type fixed -> continuous
- joint brl_final_track_joint: axis (none) -> 0.0 1 0.0; type fixed -> continuous
- joint brl_shoulder-body: axis (none) -> 1 0.0 0.0; limit (none) -> lower=-1.57075 upper=1.57075 effort=1000.0 velocity=0.5; type fixed -> revolute
- joint brl_shoulder2-knee: axis (none) -> 0.0 1 0.0; type fixed -> continuous
- joint brl_shoulder2-shoulder: axis (none) -> 0.0 1 0.0; type fixed -> continuous
- joint fll_ankle: axis (none) -> 0.0 1 0.0; type fixed -> continuous
- joint fll_final_track_joint: axis (none) -> 0.0 1 0.0; type fixed -> continuous
- joint fll_shoulder-body: axis (none) -> 1 0.0 0.0; limit (none) -> lower=-1.57075 upper=1.57075 effort=1000.0 velocity=0.5; type fixed -> revolute
- joint fll_shoulder2-knee: axis (none) -> 0.0 1 0.0; type fixed -> continuous
- joint fll_shoulder2-shoulder: axis (none) -> 0.0 1 0.0; type fixed -> continuous
- joint frl_ankle: axis (none) -> 0.0 1 0.0; type fixed -> continuous
- joint frl_final_track_joint: axis (none) -> 0.0 1 0.0; type fixed -> continuous
- joint frl_shoulder-body: axis (none) -> 1 0.0 0.0; limit (none) -> lower=-1.57075 upper=1.57075 effort=1000.0 velocity=0.5; type fixed -> revolute
- joint frl_shoulder2-knee: axis (none) -> 0.0 1 0.0; type fixed -> continuous
- joint frl_shoulder2-shoulder: axis (none) -> 0.0 1 0.0; type fixed -> continuous
