Commit message: code refactoring using xacro

File: urdf_model/cricket_robot.xacro (robot description, xacro)
@@ -6,8 +6,6 @@
   <xacro:property name="track_length" value="0.25"/>
   <xacro:property name="body_box_size" value="0.1"/>
-  <xacro:property name="bodylen" value="0.6"/>
-  <xacro:property name="baselen" value="0.4"/>
-  <xacro:property name="wheeldiam" value="0.07"/>
-  <xacro:property name="pi" value="3.1415"/>
+  <xacro:property name="pi" value="3.1415" />
+  <xacro:property name="cyl_rad" value="0.03" />
   <material name="yellow">
     <color rgba="0.8 0.8 0 1"/>
@@ -16,4 +14,10 @@
     <color rgba="1 0 0 1"/>
   </material>
+  <xacro:macro name="default_inertial" params="mass">
+    <inertial>
+      <mass value="${mass}" />
+      <inertia ixx="1.0" ixy="0.0" ixz="0.0" iyy="1.0" iyz="0.0" izz="1.0" />
+    </inertial>
+  </xacro:macro>
   <link name="base_link">
     <visual>
@@ -56,5 +60,291 @@
     </joint>
   </xacro:macro>
-  <xacro:body_box body_side="right" origin_bb="0.2" origin_bb="0.02"/>
+  <xacro:body_box body_side="right" origin_bb="0.2" origin_bc="0.02"/>
   <xacro:body_box body_side="left" origin_bb="-0.2" origin_bc="-0.02"/>
+  <!-- ###################### -->
+  <!-- ##### RIGHT LEGS ##### -->
+  <!-- ###################### -->
+  <xacro:macro name="right_leg" params="body_side o_shoulder o_s_box o_s2_base o_s2_box o_s2_base_box o_k_box o_k_base_box o_track rpy_track">
+    <!-- * SHOULDER 1 -->
+    <link name="r_${body_side}_shoulder_cylinder">
+      <visual name="r_${body_side}_shoulder_cylinder">
+        <origin rpy="0 ${pi/2} 0" xyz="0.0 0.0 0"/>
+        <geometry>
+          <cylinder radius="${cyl_rad}" length="0.12"/>
+        </geometry>
+        <material name="yellow"/>
+      </visual>
+    </link>
+    <joint name="r_${body_side}_shoulder-body" type="revolute">
+      <axis xyz="1 0.0 0.0"/>
+      <limit effort="1000.0" lower="-1.57075" upper="1.57075" velocity="0.5"/>
+      <origin xyz="${o_shoulder} 0.0 0.0" rpy="0 0 0.0"/>
+      <parent link="right_cylinder"/>
+      <child link="r_${body_side}_shoulder_cylinder"/>
+    </joint>
+    <link name="r_${body_side}_shoulder_box">
+      <visual name="r_${body_side}_shoulder_box">
+        <origin rpy="0 0 0" xyz="${o_s_box} -0.0005 0"/>
+        <geometry>
+          <box size="0.12 0.03 0.06"/>
+        </geometry>
+        <material name="yellow"/>
+      </visual>
+    </link>
+    <joint name="r_${body_side}_shoulder_cyl-box" type="fixed">
+      <origin xyz="${- o_s_box} 0.017 0.0" rpy="0.0 0.0 0.0"/>
+      <parent link="r_${body_side}_shoulder_cylinder"/>
+      <child link="r_${body_side}_shoulder_box"/>
+    </joint>
+    <!-- * SHOULDER 2  -->
+    <link name="r_${body_side}_shoulder2_base">
+      <visual name="r_${body_side}_shoulder2_base">
+        <origin xyz="${o_s2_base} 0.0 0.0" rpy="0.0 0.0 0.0"/>
+        <geometry>
+          <box size="0.05 0.01 0.06"/>
+        </geometry>
+        <material name="yellow"/>
+      </visual>
+    </link>
+    <joint name="r_${body_side}_shoulder2-shoulder" type="continuous">
+      <axis xyz="0.0 1 0.0"/>
+      <origin xyz="0.0 0.02 0.0" rpy="0.0 0.0 0.0"/>
+      <parent link="r_${body_side}_shoulder_box"/>
+      <child link="r_${body_side}_shoulder2_base"/>
+    </joint>
+    <link name="r_${body_side}_shoulder2_box">
+      <visual name="r_${body_side}_shoulder2_box">
+        <origin xyz="${o_s2_box} 0.02 0.0" rpy="0.0 0.0 0.0"/>
+        <geometry>
+          <box size="0.11 0.05 0.06"/>
+        </geometry>
+        <material name="yellow"/>
+      </visual>
+    </link>
+    <joint name="r_${body_side}_shoulder2_base-box" type="fixed">
+      <origin xyz="${o_s2_base_box} 0.0 0.0" rpy="0.0 0.0 0.0"/>
+      <parent link="r_${body_side}_shoulder2_base"/>
+      <child link="r_${body_side}_shoulder2_box"/>
+    </joint>
+    <!-- KNEE -->
+    <link name="r_${body_side}_knee_base">
+      <visual name="r_${body_side}_knee_base">
+        <origin xyz="${- o_s_box} 0.0 0.0" rpy="0.0 0.0 0.0"/>
+        <geometry>
+          <box size="0.12 0.01 0.06"/>
+        </geometry>
+        <material name="yellow"/>
+      </visual>
+    </link>
+    <joint name="r_${body_side}_shoulder2-knee" type="continuous">
+      <axis xyz="0.0 1 0.0"/>
+      <origin xyz="0.0 0.052 0.0" rpy="0.0 0.0 0.0"/>
+      <parent link="r_${body_side}_shoulder2_box"/>
+      <child link="r_${body_side}_knee_base"/>
+    </joint>
+    <link name="r_${body_side}_knee_box">
+      <visual name="r_${body_side}_knee_box">
+        <origin xyz="${o_k_box} -0.02 0.0" rpy="0.0 0.0 0.0"/>
+        <geometry>
+          <box size="0.08 0.05 0.06"/>
+        </geometry>
+        <material name="yellow"/>
+      </visual>
+    </link>
+    <joint name="r_${body_side}_knee_base-box" type="fixed">
+      <origin xyz="${o_k_base_box} 0.0 0.0" rpy="0.0 0.0 0.0"/>
+      <parent link="r_${body_side}_knee_base"/>
+      <child link="r_${body_side}_knee_box"/>
+    </joint>
+    <!-- ANKLE & TRACK -->
+    <link name="r_${body_side}_jointed_track">
+      <visual name="r_${body_side}_jointed_track">
+        <origin xyz="0.0 0.0 0.0" rpy="0.0 1.57075 1.57075"/>
+        <geometry>
+          <cylinder radius="${cyl_rad}" length="0.05"/>
+        </geometry>
+        <material name="yellow"/>
+      </visual>
+    </link>
+    <joint name="r_${body_side}_ankle" type="continuous">
+      <axis xyz="0.0 1 0.0"/>
+      <origin xyz="0.0 0.032 0.0" rpy="0.0 0.0 0.0"/>
+      <parent link="r_${body_side}_knee_box"/>
+      <child link="r_${body_side}_jointed_track"/>
+    </joint>
+    <link name="r_${body_side}_track">
+      <visual name="r_${body_side}_track">
+        <origin xyz="0.0 0.0 0.0" rpy="0.0 0.0 0.0"/>
+        <geometry>
+          <box size="0.190 0.05 0.06"/>
+        </geometry>
+        <material name="yellow"/>
+      </visual>
+    </link>
+    <joint name="r_${body_side}_jointed_track-track" type="fixed">
+      <origin xyz="0.095 0.0 0.0" rpy="0.0 ${rpy_track} 0.0"/>
+      <parent link="r_${body_side}_jointed_track"/>
+      <child link="r_${body_side}_track"/>
+    </joint>
+    <link name="r_${body_side}_ends_track">
+      <visual name="r_${body_side}_ends_track">
+        <origin xyz="0.0 0.0 0.0" rpy="0.0 1.57075 1.57075"/>
+        <geometry>
+          <cylinder radius="${cyl_rad}" length="0.05"/>
+        </geometry>
+        <material name="yellow"/>
+      </visual>
+    </link>
+    <joint name="r_${body_side}_final_track_joint" type="continuous">
+      <axis xyz="0.0 1 0.0"/>
+      <origin xyz="${o_track} 0.0 0.0" rpy="0.0 0.0 0.0"/>
+      <parent link="r_${body_side}_track"/>
+      <child link="r_${body_side}_ends_track"/>
+    </joint>
+  </xacro:macro>
+  <xacro:right_leg body_side="front" o_shoulder="0.12" o_s_box="-0.05" o_s2_base="-0.015" o_s2_box="0.045" o_s2_base_box="-0.14" o_k_box="-0.03" o_k_base_box="0.18" o_track="0.095" rpy_track="0.0"/>
+  <xacro:right_leg body_side="back" o_shoulder="-0.12" o_s_box="0.05" o_s2_base="0.015" o_s2_box="-0.045" o_s2_base_box="0.14" o_k_box="0.03" o_k_base_box="-0.18" o_track="-0.095" rpy_track="3.1415"/>
+  <!-- ###################### -->
+  <!-- ##### LEFT LEGS ##### -->
+  <!-- ###################### -->
+  <xacro:macro name="left_leg" params="body_side o_shoulder o_s_box o_s2_base o_s2_box o_s2_base_box o_k_box o_k_base_box o_track rpy_track">
+    <!-- * SHOULDER 1 -->
+    <link name="l_${body_side}_shoulder_cylinder">
+      <visual name="l_${body_side}_shoulder_cylinder">
+        <origin rpy="0 ${pi/2} 0" xyz="0.0 0.0 0"/>
+        <geometry>
+          <cylinder radius="${cyl_rad}" length="0.12"/>
+        </geometry>
+        <material name="yellow"/>
+      </visual>
+    </link>
+    <joint name="l_${body_side}_shoulder-body" type="revolute">
+      <axis xyz="1 0.0 0.0"/>
+      <limit effort="1000.0" lower="-1.57075" upper="1.57075" velocity="0.5"/>
+      <origin xyz="${o_shoulder} 0.0 0.0" rpy="0 0 0.0"/>
+      <parent link="left_cylinder"/>
+      <child link="l_${body_side}_shoulder_cylinder"/>
+    </joint>
+    <link name="l_${body_side}_shoulder_box">
+      <visual name="l_${body_side}_shoulder_box">
+        <origin rpy="0 0 0" xyz=" ${o_s_box} 0.0005 0"/>
+        <geometry>
+          <box size="0.12 0.03 0.06"/>
+        </geometry>
+        <material name="yellow"/>
+      </visual>
+    </link>
+    <joint name="l_${body_side}_shoulder_cyl-box" type="fixed">
+      <origin xyz="${- o_s_box} -0.017 0.0" rpy="0.0 0.0 0.0"/>
+      <parent link="l_${body_side}_shoulder_cylinder"/>
+      <child link="l_${body_side}_shoulder_box"/>
+    </joint>
+    <!-- * SHOULDER 2  -->
+    <link name="l_${body_side}_shoulder2_base">
+      <visual name="l_${body_side}_shoulder2_base">
+        <origin xyz="${o_s2_base} 0.0 0.0" rpy="0.0 0.0 0.0"/>
+        <geometry>
+          <box size="0.05 0.01 0.06"/>
+        </geometry>
+        <material name="yellow"/>
+      </visual>
+    </link>
+    <joint name="l_${body_side}_shoulder2-shoulder" type="continuous">
+      <axis xyz="0.0 1 0.0"/>
+      <origin xyz="0.0 -0.02 0.0" rpy="0.0 0.0 0.0"/>
+      <parent link="l_${body_side}_shoulder_box"/>
+      <child link="l_${body_side}_shoulder2_base"/>
+    </joint>
+    <link name="l_${body_side}_shoulder2_box">
+      <visual name="l_${body_side}_shoulder2_box">
+        <origin xyz="${o_s2_box} -0.02 0.0" rpy="0.0 0.0 0.0"/>
+        <geometry>
+          <box size="0.11 0.05 0.06"/>
+        </geometry>
+        <material name="yellow"/>
+      </visual>
+    </link>
+    <joint name="l_${body_side}_shoulder2_base-box" type="fixed">
+      <origin xyz="${o_s2_base_box} 0.0 0.0" rpy="0.0 0.0 0.0"/>
+      <parent link="l_${body_side}_shoulder2_base"/>
+      <child link="l_${body_side}_shoulder2_box"/>
+    </joint>
+    <!-- KNEE -->
+    <link name="l_${body_side}_knee_base">
+      <visual name="l_${body_side}_knee_base">
+        <origin xyz="${- o_s_box} 0.0 0.0" rpy="0.0 0.0 0.0"/>
+        <geometry>
+          <box size="0.12 0.01 0.06"/>
+        </geometry>
+        <material name="yellow"/>
+      </visual>
+    </link>
+    <joint name="l_${body_side}_shoulder2-knee" type="continuous">
+      <axis xyz="0.0 1 0.0"/>
+      <origin xyz="0.0 -0.052 0.0" rpy="0.0 0.0 0.0"/>
+      <parent link="l_${body_side}_shoulder2_box"/>
+      <child link="l_${body_side}_knee_base"/>
+    </joint>
+    <link name="l_${body_side}_knee_box">
+      <visual name="l_${body_side}_knee_box">
+        <origin xyz="${o_k_box} 0.02 0.0" rpy="0.0 0.0 0.0"/>
+        <geometry>
+          <box size="0.08 0.05 0.06"/>
+        </geometry>
+        <material name="yellow"/>
+      </visual>
+    </link>
+    <joint name="l_${body_side}_knee_base-box" type="fixed">
+      <origin xyz="${o_k_base_box} 0.0 0.0" rpy="0.0 0.0 0.0"/>
+      <parent link="l_${body_side}_knee_base"/>
+      <child link="l_${body_side}_knee_box"/>
+    </joint>
+    <!-- ANKLE & TRACK -->
+    <link name="l_${body_side}_jointed_track">
+      <visual name="l_${body_side}_jointed_track">
+        <origin xyz="0.0 0.0 0.0" rpy="0.0 1.57075 1.57075"/>
+        <geometry>
+          <cylinder radius="${cyl_rad}" length="0.05"/>
+        </geometry>
+        <material name="yellow"/>
+      </visual>
+    </link>
+    <joint name="l_${body_side}_ankle" type="continuous">
+      <axis xyz="0.0 1 0.0"/>
+      <origin xyz="0.0 -0.032 0.0" rpy="0.0 0.0 0.0"/>
+      <parent link="l_${body_side}_knee_box"/>
+      <child link="l_${body_side}_jointed_track"/>
+    </joint>
+    <link name="l_${body_side}_track">
+      <visual name="l_${body_side}_track">
+        <origin xyz="0.0 0.0 0.0" rpy="0.0 0.0 0.0"/>
+        <geometry>
+          <box size="0.190 0.05 0.06"/>
+        </geometry>
+        <material name="yellow"/>
+      </visual>
+    </link>
+    <joint name="l_${body_side}_jointed_track-track" type="fixed">
+      <origin xyz="0.095 0.0 0.0" rpy="0.0 ${rpy_track} 0.0"/>
+      <parent link="l_${body_side}_jointed_track"/>
+      <child link="l_${body_side}_track"/>
+    </joint>
+    <link name="l_${body_side}_ends_track">
+      <visual name="l_${body_side}_ends_track">
+        <origin xyz="0.0 0.0 0.0" rpy="0.0 1.57075 1.57075"/>
+        <geometry>
+          <cylinder radius="${cyl_rad}" length="0.05"/>
+        </geometry>
+        <material name="yellow"/>
+      </visual>
+    </link>
+    <joint name="l_${body_side}_final_track_joint" type="continuous">
+      <axis xyz="0.0 1 0.0"/>
+      <origin xyz="${o_track} 0.0 0.0" rpy="0.0 0.0 0.0"/>
+      <parent link="l_${body_side}_track"/>
+      <child link="l_${body_side}_ends_track"/>
+    </joint>
+  </xacro:macro>
+  <xacro:left_leg body_side="front" o_shoulder="0.12" o_s_box="-0.05" o_s2_base="-0.015" o_s2_box="0.045" o_s2_base_box="-0.14" o_k_box="-0.03" o_k_base_box="0.18" o_track="0.095" rpy_track="0.0"/>
+  <xacro:left_leg body_side="back" o_shoulder="-0.12" o_s_box="0.05" o_s2_base="0.015" o_s2_box="-0.045" o_s2_base_box="0.14" o_k_box="0.03" o_k_base_box="-0.18" o_track="-0.095" rpy_track="3.1415"/>
 </robot>
