Commit message: collision added

File: urdf_model/cricket_robot.xacro (robot description, xacro)
@@ -27,4 +27,9 @@
       <material name="red"/>
     </visual>
+    <collision>
+      <geometry>
+        <box size="${body_length} ${body_width} ${body_height}"/>
+      </geometry>
+    </collision>
   </link>
   <!-- ###################### -->
@@ -39,4 +44,9 @@
         <material name="red"/>
       </visual>
+      <collision>
+        <geometry>
+            <box size="${body_box_size} 0.04 ${body_height}"/>
+        </geometry>
+      </collision>
     </link>
     <joint name="body_to_${body_side}_box" type="fixed">
@@ -49,8 +59,13 @@
         <origin rpy="0 ${pi/2} 0" xyz="0 0.0 0"/>
         <geometry>
-          <cylinder radius="0.03" length="0.1"/>
+          <cylinder radius="${cyl_rad}" length="0.1"/>
         </geometry>
         <material name="red"/>
       </visual>
+      <collision>
+        <geometry>
+          <cylinder radius="${cyl_rad}" length="0.1"/>
+        </geometry>
+      </collision>
     </link>
     <joint name="${body_side}_box-cylinder" type="fixed">
@@ -75,4 +90,9 @@
         <material name="yellow"/>
       </visual>
+      <collision>
+        <geometry>
+          <cylinder radius="${cyl_rad}" length="0.12"/>
+        </geometry>
+      </collision>
     </link>
     <joint name="r_${body_side}_shoulder-body" type="revolute">
@@ -91,4 +111,9 @@
         <material name="yellow"/>
       </visual>
+      <collision>
+        <geometry>
+          <box size="0.12 0.03 0.06"/>
+        </geometry>
+      </collision>
     </link>
     <joint name="r_${body_side}_shoulder_cyl-box" type="fixed">
@@ -106,4 +131,9 @@
         <material name="yellow"/>
       </visual>
+      <collision>
+        <geometry>
+          <box size="0.05 0.01 0.06"/>
+        </geometry>
+      </collision>
     </link>
     <joint name="r_${body_side}_shoulder2-shoulder" type="continuous">
@@ -121,4 +151,9 @@
         <material name="yellow"/>
       </visual>
+      <collision>
+        <geometry>
+          <box size="0.11 0.05 0.06"/>
+        </geometry>
+      </collision>
     </link>
     <joint name="r_${body_side}_shoulder2_base-box" type="fixed">
@@ -136,4 +171,9 @@
         <material name="yellow"/>
       </visual>
+      <collision>
+        <geometry>
+          <box size="0.12 0.01 0.06"/>
+        </geometry>
+      </collision>
     </link>
     <joint name="r_${body_side}_shoulder2-knee" type="continuous">
@@ -151,4 +191,9 @@
         <material name="yellow"/>
       </visual>
+      <collision>
+        <geometry>
+          <box size="0.08 0.05 0.06"/>
+        </geometry>
+      </collision>
     </link>
     <joint name="r_${body_side}_knee_base-box" type="fixed">
@@ -166,4 +211,9 @@
         <material name="yellow"/>
       </visual>
+      <collision>
+        <geometry>
+          <cylinder radius="${cyl_rad}" length="0.05"/>
+        </geometry>
+      </collision>
     </link>
     <joint name="r_${body_side}_ankle" type="continuous">
@@ -181,4 +231,9 @@
         <material name="yellow"/>
       </visual>
+      <collision>
+        <geometry>
+          <box size="0.190 0.05 0.06"/>
+        </geometry>
+      </collision>
     </link>
     <joint name="r_${body_side}_jointed_track-track" type="fixed">
@@ -195,4 +250,9 @@
         <material name="yellow"/>
       </visual>
+      <collision>
+        <geometry>
+          <cylinder radius="${cyl_rad}" length="0.05"/>
+        </geometry>
+      </collision>
     </link>
     <joint name="r_${body_side}_final_track_joint" type="continuous">
@@ -218,4 +278,9 @@
         <material name="yellow"/>
       </visual>
+      <collision>
+        <geometry>
+          <cylinder radius="${cyl_rad}" length="0.12"/>
+        </geometry>
+      </collision>
     </link>
     <joint name="l_${body_side}_shoulder-body" type="revolute">
@@ -234,4 +299,9 @@
         <material name="yellow"/>
       </visual>
+      <collision>
+        <geometry>
+          <box size="0.12 0.03 0.06"/>
+        </geometry>
+      </collision>
     </link>
     <joint name="l_${body_side}_shoulder_cyl-box" type="fixed">
@@ -249,4 +319,9 @@
         <material name="yellow"/>
       </visual>
+      <collision>
+        <geometry>
+          <box size="0.05 0.01 0.06"/>
+        </geometry>
+      </collision>
     </link>
     <joint name="l_${body_side}_shoulder2-shoulder" type="continuous">
@@ -264,4 +339,9 @@
         <material name="yellow"/>
       </visual>
+      <collision>
+        <geometry>
+          <box size="0.11 0.05 0.06"/>
+        </geometry>
+      </collision>
     </link>
     <joint name="l_${body_side}_shoulder2_base-box" type="fixed">
@@ -279,4 +359,9 @@
         <material name="yellow"/>
       </visual>
+      <collision>
+        <geometry>
+          <box size="0.12 0.01 0.06"/>
+        </geometry>
+      </collision>
     </link>
     <joint name="l_${body_side}_shoulder2-knee" type="continuous">
@@ -294,4 +379,9 @@
         <material name="yellow"/>
       </visual>
+      <collision>
+        <geometry>
+          <box size="0.08 0.05 0.06"/>
+        </geometry>
+      </collision>
     </link>
     <joint name="l_${body_side}_knee_base-box" type="fixed">
@@ -309,4 +399,9 @@
         <material name="yellow"/>
       </visual>
+      <collision>
+        <geometry>
+          <cylinder radius="${cyl_rad}" length="0.05"/>
+        </geometry>
+      </collision>
     </link>
     <joint name="l_${body_side}_ankle" type="continuous">
@@ -324,4 +419,9 @@
         <material name="yellow"/>
       </visual>
+      <collision>
+        <geometry>
+          <box size="0.190 0.05 0.06"/>
+        </geometry>
+      </collision>
     </link>
     <joint name="l_${body_side}_jointed_track-track" type="fixed">
@@ -338,4 +438,9 @@
         <material name="yellow"/>
       </visual>
+      <collision>
+        <geometry>
+          <cylinder radius="${cyl_rad}" length="0.05"/>
+        </geometry>
+      </collision>
     </link>
     <joint name="l_${body_side}_final_track_joint" type="continuous">

File: urdf_model/cricket_robot_xacro.urdf (robot description, URDF)
Before this commit: robot cricket_robot, 41 links, 40 joints
Links:
- link base_link: geometry collision box size=0.41 0.36 0.06; visual box size=0.41 0.36 0.06
- link l_back_ends_track: geometry collision cylinder length=0.05 radius=0.03; visual cylinder length=0.05 radius=0.03
- link l_back_jointed_track: geometry collision cylinder length=0.05 radius=0.03; visual cylinder length=0.05 radius=0.03
- link l_back_knee_base: geometry collision box size=0.12 0.01 0.06; visual box size=0.12 0.01 0.06
- link l_back_knee_box: geometry collision box size=0.08 0.05 0.06; visual box size=0.08 0.05 0.06
- link l_back_shoulder2_base: geometry collision box size=0.05 0.01 0.06; visual box size=0.05 0.01 0.06
- link l_back_shoulder2_box: geometry collision box size=0.11 0.05 0.06; visual box size=0.11 0.05 0.06
- link l_back_shoulder_box: geometry collision box size=0.12 0.03 0.06; visual box size=0.12 0.03 0.06
- link l_back_shoulder_cylinder: geometry collision cylinder length=0.12 radius=0.03; visual cylinder length=0.12 radius=0.03
- link l_back_track: geometry collision box size=0.190 0.05 0.06; visual box size=0.190 0.05 0.06
- link l_front_ends_track: geometry collision cylinder length=0.05 radius=0.03; visual cylinder length=0.05 radius=0.03
- link l_front_jointed_track: geometry collision cylinder length=0.05 radius=0.03; visual cylinder length=0.05 radius=0.03
- link l_front_knee_base: geometry collision box size=0.12 0.01 0.06; visual box size=0.12 0.01 0.06
- link l_front_knee_box: geometry collision box size=0.08 0.05 0.06; visual box size=0.08 0.05 0.06
- link l_front_shoulder2_base: geometry collision box size=0.05 0.01 0.06; visual box size=0.05 0.01 0.06
- link l_front_shoulder2_box: geometry collision box size=0.11 0.05 0.06; visual box size=0.11 0.05 0.06
- link l_front_shoulder_box: geometry collision box size=0.12 0.03 0.06; visual box size=0.12 0.03 0.06
- link l_front_shoulder_cylinder: geometry collision cylinder length=0.12 radius=0.03; visual cylinder length=0.12 radius=0.03
- link l_front_track: geometry collision box size=0.190 0.05 0.06; visual box size=0.190 0.05 0.06
- link left_box: geometry collision box size=0.1 0.04 0.06; visual box size=0.1 0.04 0.06
- link left_cylinder: geometry collision cylinder length=0.1 radius=0.03; visual cylinder length=0.1 radius=0.03
- link r_back_ends_track: geometry collision cylinder length=0.05 radius=0.03; visual cylinder length=0.05 radius=0.03
- link r_back_jointed_track: geometry collision cylinder length=0.05 radius=0.03; visual cylinder length=0.05 radius=0.03
- link r_back_knee_base: geometry collision box size=0.12 0.01 0.06; visual box size=0.12 0.01 0.06
- link r_back_knee_box: geometry collision box size=0.08 0.05 0.06; visual box size=0.08 0.05 0.06
- link r_back_shoulder2_base: geometry collision box size=0.05 0.01 0.06; visual box size=0.05 0.01 0.06
- link r_back_shoulder2_box: geometry collision box size=0.11 0.05 0.06; visual box size=0.11 0.05 0.06
- link r_back_shoulder_box: geometry collision box size=0.12 0.03 0.06; visual box size=0.12 0.03 0.06
- link r_back_shoulder_cylinder: geometry collision cylinder length=0.12 radius=0.03; visual cylinder length=0.12 radius=0.03
- link r_back_track: geometry collision box size=0.190 0.05 0.06; visual box size=0.190 0.05 0.06
- link r_front_ends_track: geometry collision cylinder length=0.05 radius=0.03; visual cylinder length=0.05 radius=0.03
- link r_front_jointed_track: geometry collision cylinder length=0.05 radius=0.03; visual cylinder length=0.05 radius=0.03
- link r_front_knee_base: geometry collision box size=0.12 0.01 0.06; visual box size=0.12 0.01 0.06
- link r_front_knee_box: geometry collision box size=0.08 0.05 0.06; visual box size=0.08 0.05 0.06
- link r_front_shoulder2_base: geometry collision box size=0.05 0.01 0.06; visual box size=0.05 0.01 0.06
- link r_front_shoulder2_box: geometry collision box size=0.11 0.05 0.06; visual box size=0.11 0.05 0.06
- link r_front_shoulder_box: geometry collision box size=0.12 0.03 0.06; visual box size=0.12 0.03 0.06
- link r_front_shoulder_cylinder: geometry collision cylinder length=0.12 radius=0.03; visual cylinder length=0.12 radius=0.03
- link r_front_track: geometry collision box size=0.190 0.05 0.06; visual box size=0.190 0.05 0.06
- link right_box: geometry collision box size=0.1 0.04 0.06; visual box size=0.1 0.04 0.06
- link right_cylinder: geometry collision cylinder length=0.1 radius=0.03; visual cylinder length=0.1 radius=0.03
