Commit message: added inertia in xaro model, correction in launch

File: cricket_description/urdf/cricket_robot.urdf (robot description, URDF)
Before this commit: robot cricket_robot, 41 links, 40 joints
Links:
- added link dummy_link, mass 10; collision box size=0.0 0.0 0.0; visual box size=0.0 0.0 0.0
- link l_back_knee_base: mass None -> 4
- link l_back_shoulder2_box: mass None -> 3
- link l_back_shoulder_cylinder: mass None -> 3.5
- link l_back_track: mass None -> 4.5
- link l_front_knee_base: mass None -> 4
- link l_front_shoulder2_box: mass None -> 3
- link l_front_shoulder_cylinder: mass None -> 3.5
- link l_front_track: mass None -> 4.5
- link r_back_knee_box: mass None -> 3.5
- link r_back_shoulder2_box: mass None -> 3
- link r_back_shoulder_box: mass None -> 3.5
- link r_back_track: mass None -> 4
- link r_front_knee_box: mass None -> 3.5
- link r_front_shoulder2_box: mass None -> 3
- link r_front_shoulder_box: mass None -> 3.5
- link r_front_track: mass None -> 4
Joints:
- added joint dummy_joint: type fixed, parent base_link, child dummy_link, origin xyz=0.0 0.0 0.0 rpy=0.0 0.0 0.0, axis 0.0 0.0 0.0

File: cricket_description/urdf/cricket_robot.urdf.xacro (robot description, xacro)
@@ -9,5 +9,6 @@
   <xacro:property name="cyl_rad" value="0.03" />
   <material name="yellow">
-    <color rgba="0.8 0.8 0 1"/>
+    <!-- <color rgba="0.8 0.8 0 1"/> -->
+    <color rgba="1 0 0 1"/>
   </material>
   <material name="red">
@@ -33,4 +34,26 @@
     </collision>
   </link>
+  <link name="dummy_link">
+    <visual name="">
+      <origin xyz="0.0 0.0 0.0" rpy="0.0 0.0 0.0"/>
+      <geometry>
+        <box size="${body_length} ${body_width} ${body_height}"/>
+      </geometry>
+      <material name="red"/>
+    </visual>
+    <collision>
+      <origin xyz="0.0 0.0 0.0" rpy="0.0 0.0 0.0"/>
+      <geometry>
+        <box size="0.0 0.0 0.0"/>
+      </geometry>
+    </collision>
+    <xacro:default_inertial mass="10"/>
+  </link>
+  <joint name="dummy_joint" type="fixed">
+    <origin xyz="0.0 0.0 0.0" rpy="0.0 0.0 0.0"/>
+    <parent link="base_link"/>
+    <child link="dummy_link"/>
+    <axis xyz="0.0 0.0 0.0"/>
+  </joint>
   <!-- ###################### -->
   <!-- #####  BODY  BOX ##### -->
@@ -81,5 +104,5 @@
   <!-- ###################### -->
   <xacro:macro name="right_leg" params="body_side o_shoulder o_s_box o_s2_base o_s2_box o_s2_base_box o_k_box o_k_base_box o_track rpy_track">
-    <!-- * SHOULDER 1 -->
+    <!-- SHOULDER 1 -->
     <link name="r_${body_side}_shoulder_cylinder">
       <visual name="r_${body_side}_shoulder_cylinder">
@@ -96,5 +119,5 @@
       </collision>
     </link>
-    <joint name="r_${body_side}_shoulder-body" type="revolute">
+    <!-- <joint name="r_${body_side}_shoulder-body" type="revolute">
       <axis xyz="1 0.0 0.0"/>
       <limit effort="1000.0" lower="-1.57075" upper="1.57075" velocity="0.5"/>
@@ -102,4 +125,9 @@
       <parent link="right_cylinder"/>
       <child link="r_${body_side}_shoulder_cylinder"/>
+    </joint> -->
+    <joint name="r_${body_side}_shoulder-body" type="fixed">
+      <origin xyz="${o_shoulder} 0.0 0.0" rpy="0 0 0.0"/>
+      <parent link="right_cylinder"/>
+      <child link="r_${body_side}_shoulder_cylinder"/>
     </joint>
     <link name="r_${body_side}_shoulder_box">
@@ -116,4 +144,5 @@
         </geometry>
       </collision>
+      <xacro:default_inertial mass="3.5"/>
     </link>
     <joint name="r_${body_side}_shoulder_cyl-box" type="fixed">
@@ -122,5 +151,5 @@
       <child link="r_${body_side}_shoulder_box"/>
     </joint>
-    <!-- * SHOULDER 2  -->
+    <!-- SHOULDER 2 -->
     <link name="r_${body_side}_shoulder2_base">
       <visual name="r_${body_side}_shoulder2_base">
@@ -156,4 +185,5 @@
         </geometry>
       </collision>
+      <xacro:default_inertial mass="3"/>
     </link>
     <joint name="r_${body_side}_shoulder2_base-box" type="fixed">
@@ -196,4 +226,5 @@
         </geometry>
       </collision>
+      <xacro:default_inertial mass="3.5"/>
     </link>
     <joint name="r_${body_side}_knee_base-box" type="fixed">
@@ -236,4 +267,5 @@
         </geometry>
       </collision>
+      <xacro:default_inertial mass="4"/>
     </link>
     <joint name="r_${body_side}_jointed_track-track" type="fixed">
@@ -266,8 +298,8 @@
   <xacro:right_leg body_side="back" o_shoulder="-0.12" o_s_box="0.05" o_s2_base="0.015" o_s2_box="-0.045" o_s2_base_box="0.14" o_k_box="0.03" o_k_base_box="-0.18" o_track="-0.095" rpy_track="3.1415"/>
   <!-- ###################### -->
-  <!-- ##### LEFT LEGS ##### -->
+  <!-- ##### LEFT LEGS ###### -->
   <!-- ###################### -->
   <xacro:macro name="left_leg" params="body_side o_shoulder o_s_box o_s2_base o_s2_box o_s2_base_box o_k_box o_k_base_box o_track rpy_track">
-    <!-- * SHOULDER 1 -->
+    <!-- SHOULDER 1 -->
     <link name="l_${body_side}_shoulder_cylinder">
       <visual name="l_${body_side}_shoulder_cylinder">
@@ -283,4 +315,5 @@
         </geometry>
       </collision>
+      <xacro:default_inertial mass="3.5"/>
     </link>
     <joint name="l_${body_side}_shoulder-body" type="revolute">
@@ -310,5 +343,5 @@
       <child link="l_${body_side}_shoulder_box"/>
     </joint>
-    <!-- * SHOULDER 2  -->
+    <!-- SHOULDER 2  -->
     <link name="l_${body_side}_shoulder2_base">
       <visual name="l_${body_side}_shoulder2_base">
@@ -344,4 +377,5 @@
         </geometry>
       </collision>
+      <xacro:default_inertial mass="3"/>
     </link>
     <joint name="l_${body_side}_shoulder2_base-box" type="fixed">
@@ -364,4 +398,5 @@
         </geometry>
       </collision>
+      <xacro:default_inertial mass="4"/>
     </link>
     <joint name="l_${body_side}_shoulder2-knee" type="continuous">
@@ -424,4 +459,5 @@
         </geometry>
       </collision>
+      <xacro:default_inertial mass="4.5"/>
     </link>
     <joint name="l_${body_side}_jointed_track-track" type="fixed">

File: cricket_description/urdf/fake_cricket_robot.urdf.xacro (robot description, xacro)
@@ -7,5 +7,11 @@
   <xacro:property name="baselen" value="0.4" />
   <xacro:property name="wheeldiam" value="0.07" />
+  <xacro:property name="body_height" value="0.06"/>
+  <xacro:property name="body_length" value="0.41"/>
+  <xacro:property name="body_width" value="0.36"/>
+  <xacro:property name="track_length" value="0.25"/>
+  <xacro:property name="body_box_size" value="0.1"/>
   <xacro:property name="pi" value="3.1415" />
+  <xacro:property name="cyl_rad" value="0.03" />
   <material name="blue">
     <color rgba="0 0 0.8 1"/>
@@ -26,15 +32,61 @@
     <visual>
       <geometry>
-        <cylinder radius="${width}" length="${bodylen}"/>
-      </geometry>
-      <material name="blue"/>
-    </visual>
-    <collision>
-      <geometry>
-        <cylinder radius="${width}" length="${bodylen}"/>
-      </geometry>
-    </collision>
-    <xacro:default_inertial mass="10"/>
-  </link>
+        <box size="${body_length} ${body_width} ${body_height}"/>
+      </geometry>
+      <material name="red"/>
+    </visual>
+    <collision>
+      <geometry>
+        <box size="${body_length} ${body_width} ${body_height}"/>
+      </geometry>
+    </collision>
+  </link>
+  <!-- ###################### -->
+  <!-- #####  BODY  BOX ##### -->
+  <!-- ###################### -->
+  <xacro:macro name="body_box" params="body_side origin_bb origin_bc">
+    <link name="${body_side}_box">
+      <visual>
+        <geometry>
+            <box size="${body_box_size} 0.04 ${body_height}"/>
+        </geometry>
+        <material name="red"/>
+      </visual>
+      <collision>
+        <geometry>
+            <box size="${body_box_size} 0.04 ${body_height}"/>
+        </geometry>
+      </collision>
+    </link>
+    <joint name="body_to_${body_side}_box" type="fixed">
+      <parent link="base_link"/>
+      <child link="${body_side}_box"/>
+      <origin xyz="0.0 ${origin_bb} 0.0"/>
+    </joint>
+    <link name="${body_side}_cylinder">
+      <visual name="${body_side}_cylinder">
+        <origin rpy="0 ${pi/2} 0" xyz="0 0.0 0"/>
+        <geometry>
+          <cylinder radius="${cyl_rad}" length="0.1"/>
+        </geometry>
+        <material name="red"/>
+      </visual>
+      <collision>
+        <geometry>
+          <cylinder radius="${cyl_rad}" length="0.1"/>
+        </geometry>
+      </collision>
+    </link>
+    <joint name="${body_side}_box-cylinder" type="fixed">
+      <parent link="${body_side}_box"/>
+      <child link="${body_side}_cylinder"/>
+      <origin xyz="0.0 ${origin_bc} 0.0" rpy="0.0 0.0 0.0"/>
+    </joint>
+  </xacro:macro>
+  <xacro:body_box body_side="right" origin_bb="0.2" origin_bc="0.02"/>
+  <xacro:body_box body_side="left" origin_bb="-0.2" origin_bc="-0.02"/>
+<!-- ===========================================
+===== CAZZO
+================================================ -->
   <xacro:macro name="wheel" params="prefix suffix reflect">
     <link name="${prefix}_${suffix}_wheel">
@@ -105,5 +157,5 @@
     <xacro:wheel prefix="${prefix}" suffix="back" reflect="-1"/>
   </xacro:macro>
-  <xacro:leg prefix="right" reflect="-1" />
+  <!-- <xacro:leg prefix="right" reflect="-1" /> -->
   <xacro:leg prefix="left" reflect="1" />
   <joint name="gripper_extension" type="prismatic">
