Commit message: urdf correction and display.launch

File: cricket_description/urdf/cricket_robot.urdf.xacro (robot description, xacro)
@@ -1,19 +1,16 @@
 <?xml version="1.0"?>
-<robot name="gazebo1" xmlns:xacro="http://ros.org/wiki/xacro">
-  <xacro:property name="width" value="0.2" />
-  <xacro:property name="leglen" value="0.6" />
-  <xacro:property name="polelen" value="0.2" />
-  <xacro:property name="bodylen" value="0.6" />
-  <xacro:property name="baselen" value="0.4" />
-  <xacro:property name="wheeldiam" value="0.07" />
+<robot name="cricket_robot" xmlns:xacro="http://ros.org/wiki/xacro">
+  <xacro:property name="body_height" value="0.06"/>
+  <xacro:property name="body_length" value="0.41"/>
+  <xacro:property name="body_width" value="0.36"/>
+  <xacro:property name="track_length" value="0.25"/>
+  <xacro:property name="body_box_size" value="0.1"/>
   <xacro:property name="pi" value="3.1415" />
-  <material name="blue">
-    <color rgba="0 0 0.8 1"/>
+  <xacro:property name="cyl_rad" value="0.03" />
+  <material name="yellow">
+    <color rgba="0.8 0.8 0 1"/>
   </material>
-  <material name="black">
-    <color rgba="0 0 0 1"/>
-  </material>
-  <material name="white">
-    <color rgba="1 1 1 1"/>
+  <material name="red">
+    <color rgba="1 0 0 1"/>
   </material>
   <xacro:macro name="default_inertial" params="mass">
@@ -26,191 +23,434 @@
     <visual>
       <geometry>
-        <cylinder radius="${width}" length="${bodylen}"/>
+        <box size="${body_length} ${body_width} ${body_height}"/>
       </geometry>
-      <material name="blue"/>
+      <material name="red"/>
     </visual>
     <collision>
       <geometry>
-        <cylinder radius="${width}" length="${bodylen}"/>
+        <box size="${body_length} ${body_width} ${body_height}"/>
       </geometry>
     </collision>
-    <xacro:default_inertial mass="10"/>
   </link>
-  <xacro:macro name="wheel" params="prefix suffix reflect">
-    <link name="${prefix}_${suffix}_wheel">
+  <!-- ###################### -->
+  <!-- #####  BODY  BOX ##### -->
+  <!-- ###################### -->
+  <xacro:macro name="body_box" params="body_side origin_bb origin_bc">
+    <link name="${body_side}_box">
       <visual>
-        <origin xyz="0 0 0" rpy="${pi/2} 0 0" />
-        <geometry>
-          <cylinder radius="${wheeldiam/2}" length="0.1"/>
-        </geometry>
-        <material name="black"/>
-      </visual>
-      <collision>
-        <origin xyz="0 0 0" rpy="${pi/2} 0 0" />
-        <geometry>
-          <cylinder radius="${wheeldiam/2}" length="0.1"/>
-        </geometry>
-      </collision>
-      <xacro:default_inertial mass="1"/>
-    </link>
-    <joint name="${prefix}_${suffix}_wheel_joint" type="continuous">
-      <axis xyz="0 1 0" rpy="0 0 0" />
-      <parent link="${prefix}_base"/>
-      <child link="${prefix}_${suffix}_wheel"/>
-      <origin xyz="${baselen*reflect/3} 0 -${wheeldiam/2+.05}" rpy="0 0 0"/>
+        <geometry>
+            <box size="${body_box_size} 0.04 ${body_height}"/>
+        </geometry>
+        <material name="red"/>
+      </visual>
+      <collision>
+        <geometry>
+            <box size="${body_box_size} 0.04 ${body_height}"/>
+        </geometry>
+      </collision>
+    </link>
+    <joint name="body_to_${body_side}_box" type="fixed">
+      <parent link="base_link"/>
+      <child link="${body_side}_box"/>
+      <origin xyz="0.0 ${origin_bb} 0.0"/>
+    </joint>
+    <link name="${body_side}_cylinder">
+      <visual name="${body_side}_cylinder">
+        <origin rpy="0 ${pi/2} 0" xyz="0 0.0 0"/>
+        <geometry>
+          <cylinder radius="${cyl_rad}" length="0.1"/>
+        </geometry>
+        <material name="red"/>
+      </visual>
+      <collision>
+        <geometry>
+          <cylinder radius="${cyl_rad}" length="0.1"/>
+        </geometry>
+      </collision>
+    </link>
+    <joint name="${body_side}_box-cylinder" type="fixed">
+      <parent link="${body_side}_box"/>
+      <child link="${body_side}_cylinder"/>
+      <origin xyz="0.0 ${origin_bc} 0.0" rpy="0.0 0.0 0.0"/>
     </joint>
   </xacro:macro>
-  <xacro:macro name="leg" params="prefix reflect">
-    <link name="${prefix}_leg">
-      <visual>
-        <geometry>
-          <box size="${leglen} 0.1 0.2"/>
-        </geometry>
-        <origin xyz="0 0 -${leglen/2}" rpy="0 ${pi/2} 0"/>
-        <material name="white"/>
-      </visual>
-      <collision>
-        <geometry>
-          <box size="${leglen} 0.1 0.2"/>
-        </geometry>
-        <origin xyz="0 0 -${leglen/2}" rpy="0 ${pi/2} 0"/>
-      </collision>
-      <xacro:default_inertial mass="10"/>
-    </link>
-    <joint name="base_to_${prefix}_leg" type="fixed">
-      <parent link="base_link"/>
-      <child link="${prefix}_leg"/>
-      <origin xyz="0 ${reflect*(width+.02)} 0.25" />
-    </joint>
-    <link name="${prefix}_base">
-      <visual>
-        <geometry>
-          <box size="${baselen} 0.1 0.1"/>
-        </geometry>
-        <material name="white"/>
-      </visual>
-      <collision>
-        <geometry>
-          <box size="${baselen} 0.1 0.1"/>
-        </geometry>
-      </collision>
-      <xacro:default_inertial mass="10"/>
-    </link>
-    <joint name="${prefix}_base_joint" type="fixed">
-      <parent link="${prefix}_leg"/>
-      <child link="${prefix}_base"/>
-      <origin xyz="0 0 ${-leglen}" />
-    </joint>
-    <xacro:wheel prefix="${prefix}" suffix="front" reflect="1"/>
-    <xacro:wheel prefix="${prefix}" suffix="back" reflect="-1"/>
+  <xacro:body_box body_side="right" origin_bb="0.2" origin_bc="0.02"/>
+  <xacro:body_box body_side="left" origin_bb="-0.2" origin_bc="-0.02"/>
+  <!-- ###################### -->
+  <!-- ##### RIGHT LEGS ##### -->
+  <!-- ###################### -->
+  <xacro:macro name="right_leg" params="body_side o_shoulder o_s_box o_s2_base o_s2_box o_s2_base_box o_k_box o_k_base_box o_track rpy_track">
+    <!-- * SHOULDER 1 -->
+    <link name="r_${body_side}_shoulder_cylinder">
+      <visual name="r_${body_side}_shoulder_cylinder">
+        <origin rpy="0 ${pi/2} 0" xyz="0.0 0.0 0"/>
+        <geometry>
+          <cylinder radius="${cyl_rad}" length="0.12"/>
+        </geometry>
+        <material name="yellow"/>
+      </visual>
+      <collision>
+        <geometry>
+          <cylinder radius="${cyl_rad}" length="0.12"/>
+        </geometry>
+      </collision>
+    </link>
+    <joint name="r_${body_side}_shoulder-body" type="revolute">
+      <axis xyz="1 0.0 0.0"/>
+      <limit effort="1000.0" lower="-1.57075" upper="1.57075" velocity="0.5"/>
+      <origin xyz="${o_shoulder} 0.0 0.0" rpy="0 0 0.0"/>
+      <parent link="right_cylinder"/>
+      <child link="r_${body_side}_shoulder_cylinder"/>
+    </joint>
+    <link name="r_${body_side}_shoulder_box">
+      <visual name="r_${body_side}_shoulder_box">
+        <origin rpy="0 0 0" xyz="${o_s_box} -0.0005 0"/>
+        <geometry>
+          <box size="0.12 0.03 0.06"/>
+        </geometry>
+        <material name="yellow"/>
+      </visual>
+      <collision>
+        <geometry>
+          <box size="0.12 0.03 0.06"/>
+        </geometry>
+      </collision>
+    </link>
+    <joint name="r_${body_side}_shoulder_cyl-box" type="fixed">
+      <origin xyz="${- o_s_box} 0.017 0.0" rpy="0.0 0.0 0.0"/>
+      <parent link="r_${body_side}_shoulder_cylinder"/>
+      <child link="r_${body_side}_shoulder_box"/>
+    </joint>
+    <!-- * SHOULDER 2  -->
+    <link name="r_${body_side}_shoulder2_base">
+      <visual name="r_${body_side}_shoulder2_base">
+        <origin xyz="${o_s2_base} 0.0 0.0" rpy="0.0 0.0 0.0"/>
+        <geometry>
+          <box size="0.05 0.01 0.06"/>
+        </geometry>
+        <material name="yellow"/>
+      </visual>
+      <collision>
+        <geometry>
+          <box size="0.05 0.01 0.06"/>
+        </geometry>
+      </collision>
+    </link>
+    <joint name="r_${body_side}_shoulder2-shoulder" type="continuous">
+      <axis xyz="0.0 1 0.0"/>
+      <origin xyz="0.0 0.02 0.0" rpy="0.0 0.0 0.0"/>
+      <parent link="r_${body_side}_shoulder_box"/>
+      <child link="r_${body_side}_shoulder2_base"/>
+    </joint>
+    <link name="r_${body_side}_shoulder2_box">
+      <visual name="r_${body_side}_shoulder2_box">
+        <origin xyz="${o_s2_box} 0.02 0.0" rpy="0.0 0.0 0.0"/>
+        <geometry>
+          <box size="0.11 0.05 0.06"/>
+        </geometry>
+        <material name="yellow"/>
+      </visual>
+      <collision>
+        <geometry>
+          <box size="0.11 0.05 0.06"/>
+        </geometry>
+      </collision>
+    </link>
+    <joint name="r_${body_side}_shoulder2_base-box" type="fixed">
+      <origin xyz="${o_s2_base_box} 0.0 0.0" rpy="0.0 0.0 0.0"/>
+      <parent link="r_${body_side}_shoulder2_base"/>
+      <child link="r_${body_side}_shoulder2_box"/>
+    </joint>
+    <!-- KNEE -->
+    <link name="r_${body_side}_knee_base">
+      <visual name="r_${body_side}_knee_base">
+        <origin xyz="${- o_s_box} 0.0 0.0" rpy="0.0 0.0 0.0"/>
+        <geometry>
+          <box size="0.12 0.01 0.06"/>
+        </geometry>
+        <material name="yellow"/>
+      </visual>
+      <collision>
+        <geometry>
+          <box size="0.12 0.01 0.06"/>
+        </geometry>
+      </collision>
+    </link>
+    <joint name="r_${body_side}_shoulder2-knee" type="continuous">
+      <axis xyz="0.0 1 0.0"/>
+      <origin xyz="0.0 0.052 0.0" rpy="0.0 0.0 0.0"/>
+      <parent link="r_${body_side}_shoulder2_box"/>
+      <child link="r_${body_side}_knee_base"/>
+    </joint>
+    <link name="r_${body_side}_knee_box">
+      <visual name="r_${body_side}_knee_box">
+        <origin xyz="${o_k_box} -0.02 0.0" rpy="0.0 0.0 0.0"/>
+        <geometry>
+          <box size="0.08 0.05 0.06"/>
+        </geometry>
+        <material name="yellow"/>
+      </visual>
+      <collision>
+        <geometry>
+          <box size="0.08 0.05 0.06"/>
+        </geometry>
+      </collision>
+    </link>
+    <joint name="r_${body_side}_knee_base-box" type="fixed">
+      <origin xyz="${o_k_base_box} 0.0 0.0" rpy="0.0 0.0 0.0"/>
+      <parent link="r_${body_side}_knee_base"/>
+      <child link="r_${body_side}_knee_box"/>
+    </joint>
+    <!-- ANKLE & TRACK -->
+    <link name="r_${body_side}_jointed_track">
+      <visual name="r_${body_side}_jointed_track">
+        <origin xyz="0.0 0.0 0.0" rpy="0.0 1.57075 1.57075"/>
+        <geometry>
+          <cylinder radius="${cyl_rad}" length="0.05"/>
+        </geometry>
+        <material name="yellow"/>
+      </visual>
+      <collision>
+        <geometry>
+          <cylinder radius="${cyl_rad}" length="0.05"/>
+        </geometry>
+      </collision>
+    </link>
+    <joint name="r_${body_side}_ankle" type="continuous">
+      <axis xyz="0.0 1 0.0"/>
+      <origin xyz="0.0 0.032 0.0" rpy="0.0 0.0 0.0"/>
+      <parent link="r_${body_side}_knee_box"/>
+      <child link="r_${body_side}_jointed_track"/>
+    </joint>
+    <link name="r_${body_side}_track">
+      <visual name="r_${body_side}_track">
+        <origin xyz="0.0 0.0 0.0" rpy="0.0 0.0 0.0"/>
+        <geometry>
+          <box size="0.190 0.05 0.06"/>
+        </geometry>
+        <material name="yellow"/>
+      </visual>
+      <collision>
+        <geometry>
+          <box size="0.190 0.05 0.06"/>
+        </geometry>
+      </collision>
+    </link>
+    <joint name="r_${body_side}_jointed_track-track" type="fixed">
+      <origin xyz="0.095 0.0 0.0" rpy="0.0 ${rpy_track} 0.0"/>
+      <parent link="r_${body_side}_jointed_track"/>
+      <child link="r_${body_side}_track"/>
+    </joint>
+    <link name="r_${body_side}_ends_track">
+      <visual name="r_${body_side}_ends_track">
+        <origin xyz="0.0 0.0 0.0" rpy="0.0 1.57075 1.57075"/>
+        <geometry>
+          <cylinder radius="${cyl_rad}" length="0.05"/>
+        </geometry>
+        <material name="yellow"/>
+      </visual>
+      <collision>
+        <geometry>
+          <cylinder radius="${cyl_rad}" length="0.05"/>
+        </geometry>
+      </collision>
+    </link>
+    <joint name="r_${body_side}_final_track_joint" type="continuous">
+      <axis xyz="0.0 1 0.0"/>
+      <origin xyz="${o_track} 0.0 0.0" rpy="0.0 0.0 0.0"/>
+      <parent link="r_${body_side}_track"/>
+      <child link="r_${body_side}_ends_track"/>
+    </joint>
   </xacro:macro>
-  <xacro:leg prefix="right" reflect="-1" />
-  <xacro:leg prefix="left" reflect="1" />
-  <joint name="gripper_extension" type="prismatic">
-    <parent link="base_link"/>
-    <child link="gripper_pole"/>
-    <limit effort="1000.0" lower="-${width*2-.02}" upper="0" velocity="0.5"/>
-    <origin rpy="0 0 0" xyz="${width-.01} 0 0.2"/>
-  </joint>
-  <link name="gripper_pole">
-    <visual>
-      <geometry>
-        <cylinder length="${polelen}" radius="0.01"/>
-      </geometry>
-      <origin xyz="${polelen/2} 0 0" rpy="0 ${pi/2} 0 "/>
-    </visual>
-    <collision>
-      <geometry>
-        <cylinder length="${polelen}" radius="0.01"/>
-      </geometry>
-      <origin xyz="${polelen/2} 0 0" rpy="0 ${pi/2} 0 "/>
-    </collision>
-    <xacro:default_inertial mass="0.05"/>
-  </link>
-  <xacro:macro name="gripper" params="prefix reflect">
-    <joint name="${prefix}_gripper_joint" type="revolute">
-      <axis xyz="0 0 ${reflect}"/>
-      <limit effort="1000.0" lower="0.0" upper="0.548" velocity="0.5"/>
-      <origin rpy="0 0 0" xyz="${polelen} ${reflect*0.01} 0"/>
-      <parent link="gripper_pole"/>
-      <child link="${prefix}_gripper"/>
-    </joint>
-    <link name="${prefix}_gripper">
-      <visual>
-        <origin rpy="${(reflect-1)/2*pi} 0 0" xyz="0 0 0"/>
-        <geometry>
-          <mesh filename="package://urdf_tutorial/meshes/l_finger.dae"/>
-        </geometry>
-      </visual>
-      <collision>
-        <geometry>
-          <mesh filename="package://urdf_tutorial/meshes/l_finger.dae"/>
-        </geometry>
-        <origin rpy="${(reflect-1)/2*pi} 0 0" xyz="0 0 0"/>
-      </collision>
-      <xacro:default_inertial mass="0.05"/>
-    </link>
-    <joint name="${prefix}_tip_joint" type="fixed">
-      <parent link="${prefix}_gripper"/>
-      <child link="${prefix}_tip"/>
-    </joint>
-    <link name="${prefix}_tip">
-      <visual>
-        <origin rpy="${(reflect-1)/2*pi} 0 0" xyz="0.09137 0.00495 0"/>
-        <geometry>
-          <mesh filename="package://urdf_tutorial/meshes/l_finger_tip.dae"/>
-        </geometry>
-      </visual>
-      <collision>
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
Commit message: let's add inertias everywhere

File: cricket_description/urdf/cricket_robot.urdf.xacro (robot description, xacro)
@@ -91,4 +91,5 @@
         </geometry>
       </collision>
+      <xacro:default_inertial mass="0.5"/>
     </link>
     <joint name="${body_side}_box-cylinder" type="fixed">
@@ -118,6 +119,7 @@
         </geometry>
       </collision>
-    </link>
-    <!-- <joint name="r_${body_side}_shoulder-body" type="revolute">
+      <xacro:default_inertial mass="0.5"/>
+    </link>
+    <joint name="r_${body_side}_shoulder-body" type="revolute">
       <axis xyz="1 0.0 0.0"/>
       <limit effort="1000.0" lower="-1.57075" upper="1.57075" velocity="0.5"/>
@@ -125,10 +127,10 @@
       <parent link="right_cylinder"/>
       <child link="r_${body_side}_shoulder_cylinder"/>
-    </joint> -->
-    <joint name="r_${body_side}_shoulder-body" type="fixed">
+    </joint>
+    <!-- <joint name="r_${body_side}_shoulder-body" type="fixed">
       <origin xyz="${o_shoulder} 0.0 0.0" rpy="0 0 0.0"/>
       <parent link="right_cylinder"/>
       <child link="r_${body_side}_shoulder_cylinder"/>
-    </joint>
+    </joint> -->
     <link name="r_${body_side}_shoulder_box">
       <visual name="r_${body_side}_shoulder_box">
