Commit message: added movements in gazebo -> problem with whels

File: cricket_description/urdf/cricket_robot.urdf.xacro (robot description, xacro)
@@ -9,6 +9,5 @@
   <xacro:property name="cyl_rad" value="0.03" />
   <material name="yellow">
-    <!-- <color rgba="0.8 0.8 0 1"/> -->
-    <color rgba="1 0 0 1"/>
+    <color rgba="0.8 0.8 0 1"/>
   </material>
   <material name="red">
@@ -21,4 +20,5 @@
     </inertial>
   </xacro:macro>
+  <!-- main body -->
   <link name="base_link">
     <visual>
@@ -87,4 +87,5 @@
       </visual>
       <collision>
+        <origin rpy="0 ${pi/2} 0" xyz="0 0.0 0"/>
         <geometry>
           <cylinder radius="${cyl_rad}" length="0.1"/>
@@ -93,5 +94,5 @@
       <xacro:default_inertial mass="0.5"/>
     </link>
-    <joint name="${body_side}_box-cylinder" type="fixed">
+    <joint name="${body_side}_box_to_cylinder" type="fixed">
       <parent link="${body_side}_box"/>
       <child link="${body_side}_cylinder"/>
@@ -115,4 +116,5 @@
       </visual>
       <collision>
+        <origin rpy="0 ${pi/2} 0" xyz="0.0 0.0 0"/>
         <geometry>
           <cylinder radius="${cyl_rad}" length="0.12"/>
@@ -121,5 +123,5 @@
       <xacro:default_inertial mass="0.5"/>
     </link>
-    <joint name="r_${body_side}_shoulder-body" type="revolute">
+    <joint name="r_${body_side}_shoulder_to_body" type="revolute">
       <axis xyz="1 0.0 0.0"/>
       <limit effort="1000.0" lower="-1.57075" upper="1.57075" velocity="0.5"/>
@@ -127,10 +129,16 @@
       <parent link="right_cylinder"/>
       <child link="r_${body_side}_shoulder_cylinder"/>
-    </joint>
-    <!-- <joint name="r_${body_side}_shoulder-body" type="fixed">
-      <origin xyz="${o_shoulder} 0.0 0.0" rpy="0 0 0.0"/>
-      <parent link="right_cylinder"/>
-      <child link="r_${body_side}_shoulder_cylinder"/>
-    </joint> -->
+      <limit effort="30" velocity="1.0"/>
+      <dynamics damping="0.0" friction="0.0"/>
+    </joint>
+    <transmission name="r_${body_side}_shoulder_to_body_trans">
+      <type>transmission_interface/SimpleTransmission</type>
+      <actuator name="$${body_side}_r_shoulder_to_body_motor">
+        <mechanicalReduction>1</mechanicalReduction>
+      </actuator>
+      <joint name="r_${body_side}_shoulder_to_body">
+        <hardwareInterface>hardware_interface/PositionJointInterface</hardwareInterface>
+      </joint>
+    </transmission>
     <link name="r_${body_side}_shoulder_box">
       <visual name="r_${body_side}_shoulder_box">
@@ -142,4 +150,5 @@
       </visual>
       <collision>
+        <origin rpy="0 0 0" xyz="${o_s_box} -0.0005 0"/>
         <geometry>
           <box size="0.12 0.03 0.06"/>
@@ -148,5 +157,5 @@
       <xacro:default_inertial mass="3.5"/>
     </link>
-    <joint name="r_${body_side}_shoulder_cyl-box" type="fixed">
+    <joint name="r_${body_side}_shoulder_cyl_to_box" type="fixed">
       <origin xyz="${- o_s_box} 0.017 0.0" rpy="0.0 0.0 0.0"/>
       <parent link="r_${body_side}_shoulder_cylinder"/>
@@ -163,15 +172,28 @@
       </visual>
       <collision>
+        <origin xyz="${o_s2_base} 0.0 0.0" rpy="0.0 0.0 0.0"/>
         <geometry>
           <box size="0.05 0.01 0.06"/>
         </geometry>
       </collision>
-    </link>
-    <joint name="r_${body_side}_shoulder2-shoulder" type="continuous">
+      <xacro:default_inertial mass="0.5"/>
+    </link>
+    <joint name="r_${body_side}_shoulder2_to_shoulder" type="continuous">
       <axis xyz="0.0 1 0.0"/>
       <origin xyz="0.0 0.02 0.0" rpy="0.0 0.0 0.0"/>
       <parent link="r_${body_side}_shoulder_box"/>
       <child link="r_${body_side}_shoulder2_base"/>
-    </joint>
+      <limit effort="30" velocity="1.0"/>
+      <dynamics damping="0.0" friction="0.0"/>
+    </joint>
+    <transmission name="r_${body_side}_shoulder2_to_shoulder_trans">
+      <type>transmission_interface/SimpleTransmission</type>
+      <actuator name="${body_side}_$_shoulder2_to_shoulder_motor">
+        <mechanicalReduction>1</mechanicalReduction>
+      </actuator>
+      <joint name="r_${body_side}_shoulder2_to_shoulder">
+        <hardwareInterface>hardware_interface/PositionJointInterface</hardwareInterface>
+      </joint>
+    </transmission>
     <link name="r_${body_side}_shoulder2_box">
       <visual name="r_${body_side}_shoulder2_box">
@@ -183,4 +205,5 @@
       </visual>
       <collision>
+        <origin xyz="${o_s2_box} 0.02 0.0" rpy="0.0 0.0 0.0"/>
         <geometry>
           <box size="0.11 0.05 0.06"/>
@@ -189,5 +212,5 @@
       <xacro:default_inertial mass="3"/>
     </link>
-    <joint name="r_${body_side}_shoulder2_base-box" type="fixed">
+    <joint name="r_${body_side}_shoulder2_base_to_box" type="fixed">
       <origin xyz="${o_s2_base_box} 0.0 0.0" rpy="0.0 0.0 0.0"/>
       <parent link="r_${body_side}_shoulder2_base"/>
@@ -204,15 +227,28 @@
       </visual>
       <collision>
+        <origin xyz="${- o_s_box} 0.0 0.0" rpy="0.0 0.0 0.0"/>
         <geometry>
           <box size="0.12 0.01 0.06"/>
         </geometry>
       </collision>
-    </link>
-    <joint name="r_${body_side}_shoulder2-knee" type="continuous">
+      <xacro:default_inertial mass="0.5"/>
+    </link>
+    <joint name="r_${body_side}_shoulder2_to_knee" type="continuous">
       <axis xyz="0.0 1 0.0"/>
       <origin xyz="0.0 0.052 0.0" rpy="0.0 0.0 0.0"/>
       <parent link="r_${body_side}_shoulder2_box"/>
       <child link="r_${body_side}_knee_base"/>
-    </joint>
+      <limit effort="30" velocity="1.0"/>
+      <dynamics damping="0.0" friction="0.0"/>
+    </joint>
+    <transmission name="r_${body_side}_shoulder2_to_knee_trans">
+      <type>transmission_interface/SimpleTransmission</type>
+      <actuator name="${body_side}_r_shoulder2_to_knee_motor">
+        <mechanicalReduction>1</mechanicalReduction>
+      </actuator>
+      <joint name="r_${body_side}_shoulder2_to_knee">
+        <hardwareInterface>hardware_interface/PositionJointInterface</hardwareInterface>
+      </joint>
+    </transmission>
     <link name="r_${body_side}_knee_box">
       <visual name="r_${body_side}_knee_box">
@@ -224,4 +260,5 @@
       </visual>
       <collision>
+        <origin xyz="${o_k_box} -0.02 0.0" rpy="0.0 0.0 0.0"/>
         <geometry>
           <box size="0.08 0.05 0.06"/>
@@ -230,5 +267,5 @@
       <xacro:default_inertial mass="3.5"/>
     </link>
-    <joint name="r_${body_side}_knee_base-box" type="fixed">
+    <joint name="r_${body_side}_knee_base_to_box" type="fixed">
       <origin xyz="${o_k_base_box} 0.0 0.0" rpy="0.0 0.0 0.0"/>
       <parent link="r_${body_side}_knee_base"/>
@@ -245,8 +282,10 @@
       </visual>
       <collision>
-        <geometry>
-          <cylinder radius="${cyl_rad}" length="0.05"/>
-        </geometry>
-      </collision>
+        <origin xyz="0.0 0.0 0.0" rpy="0.0 1.57075 1.57075"/>
+        <geometry>
+          <cylinder radius="${cyl_rad}" length="0.05"/>
+        </geometry>
+      </collision>
+      <xacro:default_inertial mass="0.5"/>
     </link>
     <joint name="r_${body_side}_ankle" type="continuous">
@@ -255,5 +294,16 @@
       <parent link="r_${body_side}_knee_box"/>
       <child link="r_${body_side}_jointed_track"/>
-    </joint>
+      <limit effort="30" velocity="1.0"/>
+      <dynamics damping="0.0" friction="0.0"/>
+    </joint>
+    <transmission name="r_${body_side}_ankle_trans">
+      <type>transmission_interface/SimpleTransmission</type>
+      <actuator name="${body_side}_r_ankle_motor">
+        <mechanicalReduction>1</mechanicalReduction>
+      </actuator>
+      <joint name="r_${body_side}_ankle">
+        <hardwareInterface>hardware_interface/PositionJointInterface</hardwareInterface>
+      </joint>
+    </transmission>
     <link name="r_${body_side}_track">
       <visual name="r_${body_side}_track">
@@ -265,4 +315,5 @@
       </visual>
       <collision>
+        <origin xyz="0.0 0.0 0.0" rpy="0.0 0.0 0.0"/>
         <geometry>
           <box size="0.190 0.05 0.06"/>
@@ -271,5 +322,5 @@
       <xacro:default_inertial mass="4"/>
     </link>
-    <joint name="r_${body_side}_jointed_track-track" type="fixed">
+    <joint name="r_${body_side}_jointed_track_to_track" type="fixed">
       <origin xyz="0.095 0.0 0.0" rpy="0.0 ${rpy_track} 0.0"/>
       <parent link="r_${body_side}_jointed_track"/>
@@ -285,8 +336,10 @@
       </visual>
       <collision>
-        <geometry>
-          <cylinder radius="${cyl_rad}" length="0.05"/>
-        </geometry>
-      </collision>
+        <origin xyz="0.0 0.0 0.0" rpy="0.0 1.57075 1.57075"/>
+        <geometry>
+          <cylinder radius="${cyl_rad}" length="0.05"/>
+        </geometry>
+      </collision>
+      <xacro:default_inertial mass="0.5"/>
     </link>
     <joint name="r_${body_side}_final_track_joint" type="continuous">
@@ -295,5 +348,23 @@
       <parent link="r_${body_side}_track"/>
       <child link="r_${body_side}_ends_track"/>
-    </joint>
+      <limit effort="30" velocity="1.0"/>
+      <dynamics damping="0.0" friction="0.0"/>
+    </joint>
+    <transmission name="r_${body_side}_final_track_joint_trans">
+      <type>transmission_interface/SimpleTransmission</type>
+      <actuator name="${body_side}_r_final_track_joint_motor">
+        <mechanicalReduction>1</mechanicalReduction>
+      </actuator>
+      <joint name="r_${body_side}_final_track_joint">
+        <hardwareInterface>hardware_interface/VelocityJointInterface</hardwareInterface>
+      </joint>
+    </transmission>
+    <gazebo reference="r_${body_side}_ends_track">
+      <mu1 value="200.0"/>
+      <mu2 value="100.0"/>
+      <kp value="10000000.0" />
+      <kd value="1.0" />
+      <material>Gazebo/Grey</material>
+    </gazebo>
   </xacro:macro>
   <xacro:right_leg body_side="front" o_shoulder="0.12" o_s_box="-0.05" o_s2_base="-0.015" o_s2_box="0.045" o_s2_base_box="-0.14" o_k_box="-0.03" o_k_base_box="0.18" o_track="0.095" rpy_track="0.0"/>
@@ -313,4 +384,5 @@
       </visual>
       <collision>
+        <origin rpy="0 ${pi/2} 0" xyz="0.0 0.0 0"/>
         <geometry>
           <cylinder radius="${cyl_rad}" length="0.12"/>
@@ -319,5 +391,5 @@
       <xacro:default_inertial mass="3.5"/>
     </link>
-    <joint name="l_${body_side}_shoulder-body" type="revolute">
+    <joint name="l_${body_side}_shoulder_to_body" type="revolute">
       <axis xyz="1 0.0 0.0"/>
       <limit effort="1000.0" lower="-1.57075" upper="1.57075" velocity="0.5"/>
@@ -325,5 +397,15 @@
       <parent link="left_cylinder"/>
       <child link="l_${body_side}_shoulder_cylinder"/>
-    </joint>
+      <limit effort="30" velocity="1.0"/>
+    </joint>
+    <transmission name="l_${body_side}_shoulder_to_body_trans">
+      <type>transmission_interface/SimpleTransmission</type>
+      <actuator name="${body_side}_l_shoulder_to_body_motor">
+        <mechanicalReduction>1</mechanicalReduction>
+      </actuator>
+      <joint name="l_${body_side}_shoulder_to_body">
+        <hardwareInterface>hardware_interface/PositionJointInterface</hardwareInterface>
+      </joint>
+    </transmission>
     <link name="l_${body_side}_shoulder_box">
       <visual name="l_${body_side}_shoulder_box">
@@ -335,10 +417,12 @@
       </visual>
       <collision>
+        <origin rpy="0 0 0" xyz=" ${o_s_box} 0.0005 0"/>
         <geometry>
           <box size="0.12 0.03 0.06"/>
         </geometry>
       </collision>
-    </link>
-    <joint name="l_${body_side}_shoulder_cyl-box" type="fixed">
+      <xacro:default_inertial mass="0.5"/>
+    </link>
+    <joint name="l_${body_side}_shoulder_cyl_to_box" type="fixed">
       <origin xyz="${- o_s_box} -0.017 0.0" rpy="0.0 0.0 0.0"/>
       <parent link="l_${body_side}_shoulder_cylinder"/>
@@ -355,15 +439,27 @@
       </visual>
       <collision>
+        <origin xyz="${o_s2_base} 0.0 0.0" rpy="0.0 0.0 0.0"/>
         <geometry>
           <box size="0.05 0.01 0.06"/>
         </geometry>
       </collision>
-    </link>
-    <joint name="l_${body_side}_shoulder2-shoulder" type="continuous">
+      <xacro:default_inertial mass="0.5"/>
+    </link>
+    <joint name="l_${body_side}_shoulder2_to_shoulder" type="continuous">
       <axis xyz="0.0 1 0.0"/>
       <origin xyz="0.0 -0.02 0.0" rpy="0.0 0.0 0.0"/>
       <parent link="l_${body_side}_shoulder_box"/>
       <child link="l_${body_side}_shoulder2_base"/>
-    </joint>
+      <limit effort="30" velocity="1.0"/>
+    </joint>
+    <transmission name="l_${body_side}_shoulder2_to_shoulder_trans">
+      <type>transmission_interface/SimpleTransmission</type>
+      <actuator name="${body_side}_l_shoulder2_to_shoulder_motor">
+        <mechanicalReduction>1</mechanicalReduction>
+      </actuator>
+      <joint name="l_${body_side}_shoulder2_to_shoulder">
+        <hardwareInterface>hardware_interface/PositionJointInterface</hardwareInterface>
+      </joint>
+    </transmission>
     <link name="l_${body_side}_shoulder2_box">
       <visual name="l_${body_side}_shoulder2_box">
@@ -375,4 +471,5 @@
       </visual>
       <collision>
+        <origin xyz="${o_s2_box} -0.02 0.0" rpy="0.0 0.0 0.0"/>
         <geometry>
           <box size="0.11 0.05 0.06"/>
@@ -381,5 +478,5 @@
       <xacro:default_inertial mass="3"/>
     </link>
-    <joint name="l_${body_side}_shoulder2_base-box" type="fixed">
+    <joint name="l_${body_side}_shoulder2_base_to_box" type="fixed">
       <origin xyz="${o_s2_base_box} 0.0 0.0" rpy="0.0 0.0 0.0"/>
       <parent link="l_${body_side}_shoulder2_base"/>
@@ -396,4 +493,5 @@
       </visual>
       <collision>
+        <origin xyz="${- o_s_box} 0.0 0.0" rpy="0.0 0.0 0.0"/>
         <geometry>
           <box size="0.12 0.01 0.06"/>
@@ -402,5 +500,5 @@
       <xacro:default_inertial mass="4"/>
     </link>
-    <joint name="l_${body_side}_shoulder2-knee" type="continuous">
+    <joint name="l_${body_side}_shoulder2_to_knee" type="continuous">
       <axis xyz="0.0 1 0.0"/>
       <origin xyz="0.0 -0.052 0.0" rpy="0.0 0.0 0.0"/>
@@ -408,4 +506,13 @@
       <child link="l_${body_side}_knee_base"/>
     </joint>
+    <transmission name="l_${body_side}_shoulder2_to_knee_trans">
+      <type>transmission_interface/SimpleTransmission</type>
+      <actuator name="${body_side}_l_shoulder2_to_knee_motor">
+        <mechanicalReduction>1</mechanicalReduction>
+      </actuator>
+      <joint name="l_${body_side}_shoulder2_to_knee">
+        <hardwareInterface>hardware_interface/PositionJointInterface</hardwareInterface>
+      </joint>
+    </transmission>
     <link name="l_${body_side}_knee_box">
       <visual name="l_${body_side}_knee_box">
@@ -417,10 +524,12 @@
       </visual>
       <collision>
+        <origin xyz="${o_k_box} 0.02 0.0" rpy="0.0 0.0 0.0"/>
         <geometry>
           <box size="0.08 0.05 0.06"/>
         </geometry>
       </collision>
-    </link>
-    <joint name="l_${body_side}_knee_base-box" type="fixed">
+      <xacro:default_inertial mass="0.5"/>
+    </link>
+    <joint name="l_${body_side}_knee_base_to_box" type="fixed">
       <origin xyz="${o_k_base_box} 0.0 0.0" rpy="0.0 0.0 0.0"/>
       <parent link="l_${body_side}_knee_base"/>
@@ -437,8 +546,10 @@
       </visual>
       <collision>
-        <geometry>
-          <cylinder radius="${cyl_rad}" length="0.05"/>
-        </geometry>
-      </collision>
+        <origin xyz="0.0 0.0 0.0" rpy="0.0 1.57075 1.57075"/>
+        <geometry>
+          <cylinder radius="${cyl_rad}" length="0.05"/>
+        </geometry>
+      </collision>
+      <xacro:default_inertial mass="0.5"/>
     </link>
     <joint name="l_${body_side}_ankle" type="continuous">
@@ -448,4 +559,13 @@
       <child link="l_${body_side}_jointed_track"/>
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