Commit message: added movements in gazebo -> problem with whels

File: cricket_description/urdf/cricket_robot_xacro.urdf (robot description, URDF)
Before this commit: robot cricket_robot, 41 links, 40 joints
Links:
- added link dummy_link, mass 10; collision box size=0.0 0.0 0.0; visual box size=0.41 0.36 0.06
- link l_back_ends_track: mass None -> 0.5
- link l_back_jointed_track: mass None -> 0.5
- link l_back_knee_base: mass None -> 4
- link l_back_knee_box: mass None -> 0.5
- link l_back_shoulder2_base: mass None -> 0.5
- link l_back_shoulder2_box: mass None -> 3
- link l_back_shoulder_box: mass None -> 0.5
- link l_back_shoulder_cylinder: mass None -> 3.5
- link l_back_track: mass None -> 4.5
- link l_front_ends_track: mass None -> 0.5
- link l_front_jointed_track: mass None -> 0.5
- link l_front_knee_base: mass None -> 4
- link l_front_knee_box: mass None -> 0.5
- link l_front_shoulder2_base: mass None -> 0.5
- link l_front_shoulder2_box: mass None -> 3
- link l_front_shoulder_box: mass None -> 0.5
- link l_front_shoulder_cylinder: mass None -> 3.5
- link l_front_track: mass None -> 4.5
- link left_cylinder: mass None -> 0.5
- link r_back_ends_track: mass None -> 0.5
- link r_back_jointed_track: mass None -> 0.5
- link r_back_knee_base: mass None -> 0.5
- link r_back_knee_box: mass None -> 3.5
- link r_back_shoulder2_base: mass None -> 0.5
- link r_back_shoulder2_box: mass None -> 3
- link r_back_shoulder_box: mass None -> 3.5
- link r_back_shoulder_cylinder: mass None -> 0.5
- link r_back_track: mass None -> 4
- link r_front_ends_track: mass None -> 0.5
- link r_front_jointed_track: mass None -> 0.5
- link r_front_knee_base: mass None -> 0.5
- link r_front_knee_box: mass None -> 3.5
- link r_front_shoulder2_base: mass None -> 0.5
- link r_front_shoulder2_box: mass None -> 3
- link r_front_shoulder_box: mass None -> 3.5
- link r_front_shoulder_cylinder: mass None -> 0.5
- link r_front_track: mass None -> 4
- link right_cylinder: mass None -> 0.5
Joints:
- removed joint l_back_jointed_track-track
- removed joint l_back_knee_base-box
- removed joint l_back_shoulder-body
- removed joint l_back_shoulder2-knee
- removed joint l_back_shoulder2-shoulder
- removed joint l_back_shoulder2_base-box
- removed joint l_back_shoulder_cyl-box
- removed joint l_front_jointed_track-track
- removed joint l_front_knee_base-box
- removed joint l_front_shoulder-body
- removed joint l_front_shoulder2-knee
- removed joint l_front_shoulder2-shoulder
- removed joint l_front_shoulder2_base-box
- removed joint l_front_shoulder_cyl-box
- removed joint left_box-cylinder
- removed joint r_back_jointed_track-track
- removed joint r_back_knee_base-box
- removed joint r_back_shoulder-body
- removed joint r_back_shoulder2-knee
- removed joint r_back_shoulder2-shoulder
- removed joint r_back_shoulder2_base-box
- removed joint r_back_shoulder_cyl-box
- removed joint r_front_jointed_track-track
- removed joint r_front_knee_base-box
- removed joint r_front_shoulder-body
- removed joint r_front_shoulder2-knee
- removed joint r_front_shoulder2-shoulder
- removed joint r_front_shoulder2_base-box
- removed joint r_front_shoulder_cyl-box
- removed joint right_box-cylinder
- added joint dummy_joint: type fixed, parent base_link, child dummy_link, origin xyz=0.0 0.0 0.0 rpy=0.0 0.0 0.0, axis 0.0 0.0 0.0
- added joint l_back_jointed_track_to_track: type fixed, parent l_back_jointed_track, child l_back_track, origin xyz=0.095 0.0 0.0 rpy=0.0 3.1415 0.0
- added joint l_back_knee_base_to_box: type fixed, parent l_back_knee_base, child l_back_knee_box, origin xyz=-0.18 0.0 0.0 rpy=0.0 0.0 0.0
- added joint l_back_shoulder2_base_to_box: type fixed, parent l_back_shoulder2_base, child l_back_shoulder2_box, origin xyz=0.14 0.0 0.0 rpy=0.0 0.0 0.0
- added joint l_back_shoulder2_to_knee: type continuous, parent l_back_shoulder2_box, child l_back_knee_base, origin xyz=0.0 -0.052 0.0 rpy=0.0 0.0 0.0, axis 0.0 1 0.0
- added joint l_back_shoulder2_to_shoulder: type continuous, parent l_back_shoulder_box, child l_back_shoulder2_base, origin xyz=0.0 -0.02 0.0 rpy=0.0 0.0 0.0, axis 0.0 1 0.0, limit effort=30 velocity=1.0
- added joint l_back_shoulder_cyl_to_box: type fixed, parent l_back_shoulder_cylinder, child l_back_shoulder_box, origin xyz=-0.05 -0.017 0.0 rpy=0.0 0.0 0.0
- added joint l_back_shoulder_to_body: type revolute, parent left_cylinder, child l_back_shoulder_cylinder, origin xyz=-0.12 0.0 0.0 rpy=0 0 0.0, axis 1 0.0 0.0, limit lower=-1.57075 upper=1.57075 effort=1000.0 velocity=0.5
- added joint l_front_jointed_track_to_track: type fixed, parent l_front_jointed_track, child l_front_track, origin xyz=0.095 0.0 0.0 rpy=0.0 0.0 0.0
- added joint l_front_knee_base_to_box: type fixed, parent l_front_knee_base, child l_front_knee_box, origin xyz=0.18 0.0 0.0 rpy=0.0 0.0 0.0
- added joint l_front_shoulder2_base_to_box: type fixed, parent l_front_shoulder2_base, child l_front_shoulder2_box, origin xyz=-0.14 0.0 0.0 rpy=0.0 0.0 0.0
- added joint l_front_shoulder2_to_knee: type continuous, parent l_front_shoulder2_box, child l_front_knee_base, origin xyz=0.0 -0.052 0.0 rpy=0.0 0.0 0.0, axis 0.0 1 0.0
- added joint l_front_shoulder2_to_shoulder: type continuous, parent l_front_shoulder_box, child l_front_shoulder2_base, origin xyz=0.0 -0.02 0.0 rpy=0.0 0.0 0.0, axis 0.0 1 0.0, limit effort=30 velocity=1.0
- added joint l_front_shoulder_cyl_to_box: type fixed, parent l_front_shoulder_cylinder, child l_front_shoulder_box, origin xyz=0.05 -0.017 0.0 rpy=0.0 0.0 0.0
- added joint l_front_shoulder_to_body: type revolute, parent left_cylinder, child l_front_shoulder_cylinder, origin xyz=0.12 0.0 0.0 rpy=0 0 0.0, axis 1 0.0 0.0, limit lower=-1.57075 upper=1.57075 effort=1000.0 velocity=0.5
- added joint left_box_to_cylinder: type fixed, parent left_box, child left_cylinder, origin xyz=0.0 -0.02 0.0 rpy=0.0 0.0 0.0
- added joint r_back_jointed_track_to_track: type fixed, parent r_back_jointed_track, child r_back_track, origin xyz=0.095 0.0 0.0 rpy=0.0 3.1415 0.0
- added joint r_back_knee_base_to_box: type fixed, parent r_back_knee_base, child r_back_knee_box, origin xyz=-0.18 0.0 0.0 rpy=0.0 0.0 0.0
- added joint r_back_shoulder2_base_to_box: type fixed, parent r_back_shoulder2_base, child r_back_shoulder2_box, origin xyz=0.14 0.0 0.0 rpy=0.0 0.0 0.0
- added joint r_back_shoulder2_to_knee: type continuous, parent r_back_shoulder2_box, child r_back_knee_base, origin xyz=0.0 0.052 0.0 rpy=0.0 0.0 0.0, axis 0.0 1 0.0, limit effort=30 velocity=1.0
- added joint r_back_shoulder2_to_shoulder: type continuous, parent r_back_shoulder_box, child r_back_shoulder2_base, origin xyz=0.0 0.02 0.0 rpy=0.0 0.0 0.0, axis 0.0 1 0.0, limit effort=30 velocity=1.0
- added joint r_back_shoulder_cyl_to_box: type fixed, parent r_back_shoulder_cylinder, child r_back_shoulder_box, origin xyz=-0.05 0.017 0.0 rpy=0.0 0.0 0.0
- added joint r_back_shoulder_to_body: type revolute, parent right_cylinder, child r_back_shoulder_cylinder, origin xyz=-0.12 0.0 0.0 rpy=0 0 0.0, axis 1 0.0 0.0, limit lower=-1.57075 upper=1.57075 effort=1000.0 velocity=0.5
- added joint r_front_jointed_track_to_track: type fixed, parent r_front_jointed_track, child r_front_track, origin xyz=0.095 0.0 0.0 rpy=0.0 0.0 0.0
- added joint r_front_knee_base_to_box: type fixed, parent r_front_knee_base, child r_front_knee_box, origin xyz=0.18 0.0 0.0 rpy=0.0 0.0 0.0
- added joint r_front_shoulder2_base_to_box: type fixed, parent r_front_shoulder2_base, child r_front_shoulder2_box, origin xyz=-0.14 0.0 0.0 rpy=0.0 0.0 0.0
- added joint r_front_shoulder2_to_knee: type continuous, parent r_front_shoulder2_box, child r_front_knee_base, origin xyz=0.0 0.052 0.0 rpy=0.0 0.0 0.0, axis 0.0 1 0.0, limit effort=30 velocity=1.0
- added joint r_front_shoulder2_to_shoulder: type continuous, parent r_front_shoulder_box, child r_front_shoulder2_base, origin xyz=0.0 0.02 0.0 rpy=0.0 0.0 0.0, axis 0.0 1 0.0, limit effort=30 velocity=1.0
- added joint r_front_shoulder_cyl_to_box: type fixed, parent r_front_shoulder_cylinder, child r_front_shoulder_box, origin xyz=0.05 0.017 0.0 rpy=0.0 0.0 0.0
- added joint r_front_shoulder_to_body: type revolute, parent right_cylinder, child r_front_shoulder_cylinder, origin xyz=0.12 0.0 0.0 rpy=0 0 0.0, axis 1 0.0 0.0, limit lower=-1.57075 upper=1.57075 effort=1000.0 velocity=0.5
- added joint right_box_to_cylinder: type fixed, parent right_box, child right_cylinder, origin xyz=0.0 0.02 0.0 rpy=0.0 0.0 0.0
- joint r_back_ankle: limit (none) -> effort=30 velocity=1.0
- joint r_back_final_track_joint: limit (none) -> effort=30 velocity=1.0
- joint r_front_ankle: limit (none) -> effort=30 velocity=1.0
- joint r_front_final_track_joint: limit (none) -> effort=30 velocity=1.0

File: cricket_description/urdf/fake_cricket_robot.urdf.xacro (robot description, xacro)
@@ -1,4 +1,4 @@
 <?xml version="1.0"?>
-<robot name="gazebo1" xmlns:xacro="http://ros.org/wiki/xacro">
+<robot name="first_transmission" xmlns:xacro="http://ros.org/wiki/xacro">
   <xacro:property name="width" value="0.2" />
   <xacro:property name="leglen" value="0.6" />
@@ -7,11 +7,5 @@
   <xacro:property name="baselen" value="0.4" />
   <xacro:property name="wheeldiam" value="0.07" />
-  <xacro:property name="body_height" value="0.06"/>
-  <xacro:property name="body_length" value="0.41"/>
-  <xacro:property name="body_width" value="0.36"/>
-  <xacro:property name="track_length" value="0.25"/>
-  <xacro:property name="body_box_size" value="0.1"/>
   <xacro:property name="pi" value="3.1415" />
-  <xacro:property name="cyl_rad" value="0.03" />
   <material name="blue">
     <color rgba="0 0 0.8 1"/>
@@ -32,61 +26,15 @@
     <visual>
       <geometry>
-        <box size="${body_length} ${body_width} ${body_height}"/>
-      </geometry>
-      <material name="red"/>
-    </visual>
-    <collision>
-      <geometry>
-        <box size="${body_length} ${body_width} ${body_height}"/>
-      </geometry>
-    </collision>
-  </link>
-  <!-- ###################### -->
-  <!-- #####  BODY  BOX ##### -->
-  <!-- ###################### -->
-  <xacro:macro name="body_box" params="body_side origin_bb origin_bc">
-    <link name="${body_side}_box">
-      <visual>
-        <geometry>
-            <box size="${body_box_size} 0.04 ${body_height}"/>
-        </geometry>
-        <material name="red"/>
-      </visual>
-      <collision>
-        <geometry>
-            <box size="${body_box_size} 0.04 ${body_height}"/>
-        </geometry>
-      </collision>
-    </link>
-    <joint name="body_to_${body_side}_box" type="fixed">
-      <parent link="base_link"/>
-      <child link="${body_side}_box"/>
-      <origin xyz="0.0 ${origin_bb} 0.0"/>
-    </joint>
-    <link name="${body_side}_cylinder">
-      <visual name="${body_side}_cylinder">
-        <origin rpy="0 ${pi/2} 0" xyz="0 0.0 0"/>
-        <geometry>
-          <cylinder radius="${cyl_rad}" length="0.1"/>
-        </geometry>
-        <material name="red"/>
-      </visual>
-      <collision>
-        <geometry>
-          <cylinder radius="${cyl_rad}" length="0.1"/>
-        </geometry>
-      </collision>
-    </link>
-    <joint name="${body_side}_box-cylinder" type="fixed">
-      <parent link="${body_side}_box"/>
-      <child link="${body_side}_cylinder"/>
-      <origin xyz="0.0 ${origin_bc} 0.0" rpy="0.0 0.0 0.0"/>
-    </joint>
-  </xacro:macro>
-  <xacro:body_box body_side="right" origin_bb="0.2" origin_bc="0.02"/>
-  <xacro:body_box body_side="left" origin_bb="-0.2" origin_bc="-0.02"/>
-<!-- ===========================================
-===== CAZZO
-================================================ -->
+        <cylinder radius="${width}" length="${bodylen}"/>
+      </geometry>
+      <material name="blue"/>
+    </visual>
+    <collision>
+      <geometry>
+        <cylinder radius="${width}" length="${bodylen}"/>
+      </geometry>
+    </collision>
+    <xacro:default_inertial mass="10"/>
+  </link>
   <xacro:macro name="wheel" params="prefix suffix reflect">
     <link name="${prefix}_${suffix}_wheel">
@@ -157,5 +105,5 @@
     <xacro:wheel prefix="${prefix}" suffix="back" reflect="-1"/>
   </xacro:macro>
-  <!-- <xacro:leg prefix="right" reflect="-1" /> -->
+  <xacro:leg prefix="right" reflect="-1" />
   <xacro:leg prefix="left" reflect="1" />
   <joint name="gripper_extension" type="prismatic">
@@ -245,4 +193,15 @@
     <origin xyz="0 0 ${bodylen/2}"/>
   </joint>
+  <!-- This block connects the head_swivel joint to an actuator (motor), which informs both
+  simulation and visualization of the robot -->
+  <transmission name="head_swivel_trans">
+    <type>transmission_interface/SimpleTransmission</type>
+    <actuator name="$head_swivel_motor">
+      <mechanicalReduction>1</mechanicalReduction>
+    </actuator>
+    <joint name="head_swivel">
+      <hardwareInterface>PositionJointInterface</hardwareInterface>
+    </joint>
+  </transmission>
   <link name="box">
     <visual>

Commit message: correction in PIDs and res conflicts

File: cricket_description/urdf/cricket_robot.urdf.xacro (robot description, xacro)
@@ -617,7 +617,15 @@
       </actuator>
       <joint name="l_${body_side}_final_track_joint">
-        <hardwareInterface>hardware_interface/PositionJointInterface</hardwareInterface>
-      </joint>
-    </transmission>
+        <hardwareInterface>hardware_interface/VelocityJointInterface</hardwareInterface>
+        <!-- <hardwareInterface>hardware_interface/PositionJointInterface</hardwareInterface> -->
+      </joint>
+    </transmission>
+    <gazebo reference="r_${body_side}_ends_track">
+      <mu1 value="200.0"/>
+      <mu2 value="100.0"/>
+      <kp value="10000000.0" />
+      <kd value="1.0" />
+      <material>Gazebo/Grey</material>
+    </gazebo>
   </xacro:macro>
   <xacro:left_leg body_side="front" o_shoulder="0.12" o_s_box="-0.05" o_s2_base="-0.015" o_s2_box="0.045" o_s2_base_box="-0.14" o_k_box="-0.03" o_k_base_box="0.18" o_track="0.095" rpy_track="0.0"/>
