Commit message: cleaned xacro file

File: cricket_description/urdf/cricket_robot.urdf.xacro (robot description, xacro)
@@ -8,4 +8,13 @@
   <xacro:property name="pi" value="3.1415" />
   <xacro:property name="cyl_rad" value="0.03" />
+  <!-- Leg values -->
+  <xacro:property name="shoulder" value="0.12" />
+  <xacro:property name="s_box" value="-0.05" />
+  <xacro:property name="s2_base" value="-0.015" />
+  <xacro:property name="s2_box" value="0.045" />
+  <xacro:property name="s2_base_box" value="-0.14"/>
+  <xacro:property name="k_box" value="-0.03" />
+  <xacro:property name="k_base_box" value="0.18" />
+  <xacro:property name="track" value="0.095" />
   <material name="yellow">
     <color rgba="0.8 0.8 0 1"/>
@@ -105,5 +114,6 @@
   <!-- ##### RIGHT LEGS ##### -->
   <!-- ###################### -->
-  <xacro:macro name="right_leg" params="body_side o_shoulder o_s_box o_s2_base o_s2_box o_s2_base_box o_k_box o_k_base_box o_track rpy_track">
+  <!-- <xacro:macro name="right_leg" params="body_side shoulder s_box s2_base s2_box s2_base_box k_box k_base_box track rpy_track"> -->
+  <xacro:macro name="right_leg" params="body_side rev rpy_track">
     <!-- SHOULDER 1 -->
     <link name="r_${body_side}_shoulder_cylinder">
@@ -126,5 +136,5 @@
       <axis xyz="1 0.0 0.0"/>
       <limit effort="1000.0" lower="-1.57075" upper="1.57075" velocity="0.5"/>
-      <origin xyz="${o_shoulder} 0.0 0.0" rpy="0 0 0.0"/>
+      <origin xyz="${rev*shoulder} 0.0 0.0" rpy="0 0 0.0"/>
       <parent link="right_cylinder"/>
       <child link="r_${body_side}_shoulder_cylinder"/>
@@ -134,5 +144,5 @@
     <transmission name="r_${body_side}_shoulder_to_body_trans">
       <type>transmission_interface/SimpleTransmission</type>
-      <actuator name="$${body_side}_r_shoulder_to_body_motor">
+      <actuator name="${body_side}_r_shoulder_to_body_motor">
         <mechanicalReduction>1</mechanicalReduction>
       </actuator>
@@ -143,5 +153,5 @@
     <link name="r_${body_side}_shoulder_box">
       <visual name="r_${body_side}_shoulder_box">
-        <origin rpy="0 0 0" xyz="${o_s_box} -0.0005 0"/>
+        <origin rpy="0 0 0" xyz="${rev*s_box} -0.0005 0"/>
         <geometry>
           <box size="0.12 0.03 0.06"/>
@@ -150,5 +160,5 @@
       </visual>
       <collision>
-        <origin rpy="0 0 0" xyz="${o_s_box} -0.0005 0"/>
+        <origin rpy="0 0 0" xyz="${rev*s_box} -0.0005 0"/>
         <geometry>
           <box size="0.12 0.03 0.06"/>
@@ -158,5 +168,5 @@
     </link>
     <joint name="r_${body_side}_shoulder_cyl_to_box" type="fixed">
-      <origin xyz="${- o_s_box} 0.017 0.0" rpy="0.0 0.0 0.0"/>
+      <origin xyz="${- rev * s_box} 0.017 0.0" rpy="0.0 0.0 0.0"/>
       <parent link="r_${body_side}_shoulder_cylinder"/>
       <child link="r_${body_side}_shoulder_box"/>
@@ -165,5 +175,5 @@
     <link name="r_${body_side}_shoulder2_base">
       <visual name="r_${body_side}_shoulder2_base">
-        <origin xyz="${o_s2_base} 0.0 0.0" rpy="0.0 0.0 0.0"/>
+        <origin xyz="${rev*s2_base} 0.0 0.0" rpy="0.0 0.0 0.0"/>
         <geometry>
           <box size="0.05 0.01 0.06"/>
@@ -172,5 +182,5 @@
       </visual>
       <collision>
-        <origin xyz="${o_s2_base} 0.0 0.0" rpy="0.0 0.0 0.0"/>
+        <origin xyz="${rev*s2_base} 0.0 0.0" rpy="0.0 0.0 0.0"/>
         <geometry>
           <box size="0.05 0.01 0.06"/>
@@ -198,5 +208,5 @@
     <link name="r_${body_side}_shoulder2_box">
       <visual name="r_${body_side}_shoulder2_box">
-        <origin xyz="${o_s2_box} 0.02 0.0" rpy="0.0 0.0 0.0"/>
+        <origin xyz="${rev*s2_box} 0.02 0.0" rpy="0.0 0.0 0.0"/>
         <geometry>
           <box size="0.11 0.05 0.06"/>
@@ -205,5 +215,5 @@
       </visual>
       <collision>
-        <origin xyz="${o_s2_box} 0.02 0.0" rpy="0.0 0.0 0.0"/>
+        <origin xyz="${rev*s2_box} 0.02 0.0" rpy="0.0 0.0 0.0"/>
         <geometry>
           <box size="0.11 0.05 0.06"/>
@@ -213,5 +223,5 @@
     </link>
     <joint name="r_${body_side}_shoulder2_base_to_box" type="fixed">
-      <origin xyz="${o_s2_base_box} 0.0 0.0" rpy="0.0 0.0 0.0"/>
+      <origin xyz="${rev*s2_base_box} 0.0 0.0" rpy="0.0 0.0 0.0"/>
       <parent link="r_${body_side}_shoulder2_base"/>
       <child link="r_${body_side}_shoulder2_box"/>
@@ -220,5 +230,5 @@
     <link name="r_${body_side}_knee_base">
       <visual name="r_${body_side}_knee_base">
-        <origin xyz="${- o_s_box} 0.0 0.0" rpy="0.0 0.0 0.0"/>
+        <origin xyz="${-rev * s_box} 0.0 0.0" rpy="0.0 0.0 0.0"/>
         <geometry>
           <box size="0.12 0.01 0.06"/>
@@ -227,5 +237,5 @@
       </visual>
       <collision>
-        <origin xyz="${- o_s_box} 0.0 0.0" rpy="0.0 0.0 0.0"/>
+        <origin xyz="${-rev * s_box} 0.0 0.0" rpy="0.0 0.0 0.0"/>
         <geometry>
           <box size="0.12 0.01 0.06"/>
@@ -253,5 +263,5 @@
     <link name="r_${body_side}_knee_box">
       <visual name="r_${body_side}_knee_box">
-        <origin xyz="${o_k_box} -0.02 0.0" rpy="0.0 0.0 0.0"/>
+        <origin xyz="${rev*k_box} -0.02 0.0" rpy="0.0 0.0 0.0"/>
         <geometry>
           <box size="0.08 0.05 0.06"/>
@@ -260,5 +270,5 @@
       </visual>
       <collision>
-        <origin xyz="${o_k_box} -0.02 0.0" rpy="0.0 0.0 0.0"/>
+        <origin xyz="${rev*k_box} -0.02 0.0" rpy="0.0 0.0 0.0"/>
         <geometry>
           <box size="0.08 0.05 0.06"/>
@@ -268,5 +278,5 @@
     </link>
     <joint name="r_${body_side}_knee_base_to_box" type="fixed">
-      <origin xyz="${o_k_base_box} 0.0 0.0" rpy="0.0 0.0 0.0"/>
+      <origin xyz="${rev*k_base_box} 0.0 0.0" rpy="0.0 0.0 0.0"/>
       <parent link="r_${body_side}_knee_base"/>
       <child link="r_${body_side}_knee_box"/>
@@ -345,5 +355,5 @@
     <joint name="r_${body_side}_final_track_joint" type="continuous">
       <axis xyz="0.0 1 0.0"/>
-      <origin xyz="${o_track} 0.0 0.0" rpy="0.0 0.0 0.0"/>
+      <origin xyz="${rev*track} 0.0 0.0" rpy="0.0 0.0 0.0"/>
       <parent link="r_${body_side}_track"/>
       <child link="r_${body_side}_ends_track"/>
@@ -368,10 +378,13 @@
     </gazebo>
   </xacro:macro>
-  <xacro:right_leg body_side="front" o_shoulder="0.12" o_s_box="-0.05" o_s2_base="-0.015" o_s2_box="0.045" o_s2_base_box="-0.14" o_k_box="-0.03" o_k_base_box="0.18" o_track="0.095" rpy_track="0.0"/>
-  <xacro:right_leg body_side="back" o_shoulder="-0.12" o_s_box="0.05" o_s2_base="0.015" o_s2_box="-0.045" o_s2_base_box="0.14" o_k_box="0.03" o_k_base_box="-0.18" o_track="-0.095" rpy_track="3.1415"/>
+  <!-- <xacro:right_leg body_side="front" shoulder="0.12" s_box="0.05" s2_base="-0.015" s2_box="0.045" s2_base_box="-0.14" k_box="-0.03" k_base_box="0.18" track="0.095" rpy_track="0.0"/>
+  <xacro:right_leg body_side="back" shoulder="-0.12" s_box="0.05" s2_base="0.015" s2_box="-0.045" s2_base_box="0.14" k_box="0.03" k_base_box="-0.18" track="-0.095" rpy_track="3.1415"/> -->
+  <xacro:right_leg body_side="front" rev="1" rpy_track="0.0"/>
+  <xacro:right_leg body_side="back" rev="-1" rpy_track="3.1415"/>
   <!-- ###################### -->
   <!-- ##### LEFT LEGS ###### -->
   <!-- ###################### -->
-  <xacro:macro name="left_leg" params="body_side o_shoulder o_s_box o_s2_base o_s2_box o_s2_base_box o_k_box o_k_base_box o_track rpy_track">
+  <!-- <xacro:macro name="left_leg" params="body_side shoulder s_box s2_base s2_box s2_base_box k_box k_base_box track rpy_track"> -->
+  <xacro:macro name="left_leg" params="body_side rev rpy_track">
     <!-- SHOULDER 1 -->
     <link name="l_${body_side}_shoulder_cylinder">
@@ -394,5 +407,5 @@
       <axis xyz="1 0.0 0.0"/>
       <limit effort="1000.0" lower="-1.57075" upper="1.57075" velocity="0.5"/>
-      <origin xyz="${o_shoulder} 0.0 0.0" rpy="0 0 0.0"/>
+      <origin xyz="${rev*shoulder} 0.0 0.0" rpy="0 0 0.0"/>
       <parent link="left_cylinder"/>
       <child link="l_${body_side}_shoulder_cylinder"/>
@@ -410,5 +423,5 @@
     <link name="l_${body_side}_shoulder_box">
       <visual name="l_${body_side}_shoulder_box">
-        <origin rpy="0 0 0" xyz=" ${o_s_box} 0.0005 0"/>
+        <origin rpy="0 0 0" xyz=" ${rev*s_box} 0.0005 0"/>
         <geometry>
           <box size="0.12 0.03 0.06"/>
@@ -417,5 +430,5 @@
       </visual>
       <collision>
-        <origin rpy="0 0 0" xyz=" ${o_s_box} 0.0005 0"/>
+        <origin rpy="0 0 0" xyz=" ${rev*s_box} 0.0005 0"/>
         <geometry>
           <box size="0.12 0.03 0.06"/>
@@ -425,5 +438,5 @@
     </link>
     <joint name="l_${body_side}_shoulder_cyl_to_box" type="fixed">
-      <origin xyz="${- o_s_box} -0.017 0.0" rpy="0.0 0.0 0.0"/>
+      <origin xyz="${- rev*s_box} -0.017 0.0" rpy="0.0 0.0 0.0"/>
       <parent link="l_${body_side}_shoulder_cylinder"/>
       <child link="l_${body_side}_shoulder_box"/>
@@ -432,5 +445,5 @@
     <link name="l_${body_side}_shoulder2_base">
       <visual name="l_${body_side}_shoulder2_base">
-        <origin xyz="${o_s2_base} 0.0 0.0" rpy="0.0 0.0 0.0"/>
+        <origin xyz="${rev*s2_base} 0.0 0.0" rpy="0.0 0.0 0.0"/>
         <geometry>
           <box size="0.05 0.01 0.06"/>
@@ -439,5 +452,5 @@
       </visual>
       <collision>
-        <origin xyz="${o_s2_base} 0.0 0.0" rpy="0.0 0.0 0.0"/>
+        <origin xyz="${rev*s2_base} 0.0 0.0" rpy="0.0 0.0 0.0"/>
         <geometry>
           <box size="0.05 0.01 0.06"/>
@@ -452,4 +465,5 @@
       <child link="l_${body_side}_shoulder2_base"/>
       <limit effort="30" velocity="1.0"/>
+      <dynamics damping="0.0" friction="0.0"/>
     </joint>
     <transmission name="l_${body_side}_shoulder2_to_shoulder_trans">
@@ -464,5 +478,5 @@
     <link name="l_${body_side}_shoulder2_box">
       <visual name="l_${body_side}_shoulder2_box">
-        <origin xyz="${o_s2_box} -0.02 0.0" rpy="0.0 0.0 0.0"/>
+        <origin xyz="${rev*s2_box} -0.02 0.0" rpy="0.0 0.0 0.0"/>
         <geometry>
           <box size="0.11 0.05 0.06"/>
@@ -471,5 +485,5 @@
       </visual>
       <collision>
-        <origin xyz="${o_s2_box} -0.02 0.0" rpy="0.0 0.0 0.0"/>
+        <origin xyz="${rev*s2_box} -0.02 0.0" rpy="0.0 0.0 0.0"/>
         <geometry>
           <box size="0.11 0.05 0.06"/>
@@ -479,5 +493,5 @@
     </link>
     <joint name="l_${body_side}_shoulder2_base_to_box" type="fixed">
-      <origin xyz="${o_s2_base_box} 0.0 0.0" rpy="0.0 0.0 0.0"/>
+      <origin xyz="${rev*s2_base_box} 0.0 0.0" rpy="0.0 0.0 0.0"/>
       <parent link="l_${body_side}_shoulder2_base"/>
       <child link="l_${body_side}_shoulder2_box"/>
@@ -486,5 +500,5 @@
     <link name="l_${body_side}_knee_base">
       <visual name="l_${body_side}_knee_base">
-        <origin xyz="${- o_s_box} 0.0 0.0" rpy="0.0 0.0 0.0"/>
+        <origin xyz="${-rev*s_box} 0.0 0.0" rpy="0.0 0.0 0.0"/>
         <geometry>
           <box size="0.12 0.01 0.06"/>
@@ -493,5 +507,5 @@
       </visual>
       <collision>
-        <origin xyz="${- o_s_box} 0.0 0.0" rpy="0.0 0.0 0.0"/>
+        <origin xyz="${-rev*s_box} 0.0 0.0" rpy="0.0 0.0 0.0"/>
         <geometry>
           <box size="0.12 0.01 0.06"/>
@@ -517,5 +531,5 @@
     <link name="l_${body_side}_knee_box">
       <visual name="l_${body_side}_knee_box">
-        <origin xyz="${o_k_box} 0.02 0.0" rpy="0.0 0.0 0.0"/>
+        <origin xyz="${rev*k_box} 0.02 0.0" rpy="0.0 0.0 0.0"/>
         <geometry>
           <box size="0.08 0.05 0.06"/>
@@ -524,5 +538,5 @@
       </visual>
       <collision>
-        <origin xyz="${o_k_box} 0.02 0.0" rpy="0.0 0.0 0.0"/>
+        <origin xyz="${rev*k_box} 0.02 0.0" rpy="0.0 0.0 0.0"/>
         <geometry>
           <box size="0.08 0.05 0.06"/>
@@ -532,5 +546,5 @@
     </link>
     <joint name="l_${body_side}_knee_base_to_box" type="fixed">
-      <origin xyz="${o_k_base_box} 0.0 0.0" rpy="0.0 0.0 0.0"/>
+      <origin xyz="${rev*k_base_box} 0.0 0.0" rpy="0.0 0.0 0.0"/>
       <parent link="l_${body_side}_knee_base"/>
       <child link="l_${body_side}_knee_box"/>
@@ -607,5 +621,5 @@
     <joint name="l_${body_side}_final_track_joint" type="continuous">
       <axis xyz="0.0 1 0.0"/>
-      <origin xyz="${o_track} 0.0 0.0" rpy="0.0 0.0 0.0"/>
+      <origin xyz="${rev*track} 0.0 0.0" rpy="0.0 0.0 0.0"/>
       <parent link="l_${body_side}_track"/>
       <child link="l_${body_side}_ends_track"/>
@@ -629,6 +643,10 @@
     </gazebo>
   </xacro:macro>
-  <xacro:left_leg body_side="front" o_shoulder="0.12" o_s_box="-0.05" o_s2_base="-0.015" o_s2_box="0.045" o_s2_base_box="-0.14" o_k_box="-0.03" o_k_base_box="0.18" o_track="0.095" rpy_track="0.0"/>
-  <xacro:left_leg body_side="back" o_shoulder="-0.12" o_s_box="0.05" o_s2_base="0.015" o_s2_box="-0.045" o_s2_base_box="0.14" o_k_box="0.03" o_k_base_box="-0.18" o_track="-0.095" rpy_track="3.1415"/>
+  <!--
+  <xacro:left_leg body_side="front" shoulder="0.12" s_box="-0.05" s2_base="-0.015" s2_box="0.045" s2_base_box="-0.14" k_box="-0.03" k_base_box="0.18" track="0.095" rpy_track="0.0"/>
+  <xacro:left_leg body_side="back" shoulder="-0.12" s_box="0.05" s2_base="0.015" s2_box="-0.045" s2_base_box="0.14" k_box="0.03" k_base_box="-0.18" track="-0.095" rpy_track="3.1415"/>
+  -->
+  <xacro:left_leg body_side="front" rev="1" rpy_track="0.0"/>
+  <xacro:left_leg body_side="back" rev="-1" rpy_track="3.1415"/>
   <!-- Gazebo plugin for ROS Control -->
   <gazebo>

Commit message: added commands and corrected wheels

File: cricket_description/urdf/cricket_robot.urdf.xacro (robot description, xacro)
@@ -291,12 +291,12 @@
         <origin xyz="0.0 0.0 0.0" rpy="0.0 1.57075 1.57075"/>
         <geometry>
-          <cylinder radius="${cyl_rad}" length="0.05"/>
-        </geometry>
-        <material name="yellow"/>
-      </visual>
-      <collision>
-        <origin xyz="0.0 0.0 0.0" rpy="0.0 1.57075 1.57075"/>
-        <geometry>
-          <cylinder radius="${cyl_rad}" length="0.05"/>
+          <cylinder radius="${cyl_rad - cyl_rad/2}" length="0.05"/>
+        </geometry>
+        <material name="yellow"/>
+      </visual>
+      <collision>
+        <origin xyz="0.0 0.0 0.0" rpy="0.0 1.57075 1.57075"/>
+        <geometry>
+          <cylinder radius="${cyl_rad - cyl_rad/2}" length="0.05"/>
         </geometry>
       </collision>
@@ -320,9 +320,48 @@
       </joint>
     </transmission>
-    <link name="r_${body_side}_track">
+    <!--wheels-->
+    <link name="r_${body_side}_starts_track">
+      <visual name="r_${body_side}_starts_track">
+        <origin xyz="0.0 0.0 0.0" rpy="0.0 1.57075 1.57075"/>
+        <geometry>
+          <cylinder radius="${cyl_rad}" length="0.05"/>
+        </geometry>
+        <material name="yellow"/>
+      </visual>
+      <collision>
+        <origin xyz="0.0 0.0 0.0" rpy="0.0 1.57075 1.57075"/>
+        <geometry>
+          <cylinder radius="${cyl_rad}" length="0.05"/>
+        </geometry>
+      </collision>
+      <xacro:default_inertial mass="0.5"/>
+    </link>
+    <joint name="r_${body_side}_begin_track_joint" type="continuous">
+      <axis xyz="0.0 1 0.0"/>
+      <origin xyz="0.0 0 0.0" rpy="0.0 0.0 0.0"/>
+      <parent link="r_${body_side}_jointed_track"/>
+      <child link="r_${body_side}_starts_track"/>
+    </joint>
+    <transmission name="r_${body_side}_begin_track_joint_trans">
+      <type>transmission_interface/SimpleTransmission</type>
+      <actuator name="${body_side}_r_begin_track_joint_motor">
+        <mechanicalReduction>1</mechanicalReduction>
+      </actuator>
+      <joint name="r_${body_side}_begin_track_joint">
+        <hardwareInterface>hardware_interface/PositionJointInterface</hardwareInterface>
+      </joint>
+    </transmission>
+    <gazebo reference="r_${body_side}_starts_track">
+      <mu1 value="200.0"/>
+      <mu2 value="100.0"/>
+      <kp value="10000000.0" />
+      <kd value="1.0" />
+      <material>Gazebo/Grey</material>
+    </gazebo>
+    <link name="r_${body_side}_track"> <!-- Between the two wheels -->
       <visual name="r_${body_side}_track">
         <origin xyz="0.0 0.0 0.0" rpy="0.0 0.0 0.0"/>
         <geometry>
-          <box size="0.190 0.05 0.06"/>
+          <box size="0.190 0.04 0.06"/>
         </geometry>
         <material name="yellow"/>
@@ -331,5 +370,5 @@
         <origin xyz="0.0 0.0 0.0" rpy="0.0 0.0 0.0"/>
         <geometry>
-          <box size="0.190 0.05 0.06"/>
+          <box size="0.190 0.04 0.06"/>
         </geometry>
       </collision>
@@ -559,17 +598,17 @@
         <origin xyz="0.0 0.0 0.0" rpy="0.0 1.57075 1.57075"/>
         <geometry>
-          <cylinder radius="${cyl_rad}" length="0.05"/>
-        </geometry>
-        <material name="yellow"/>
-      </visual>
-      <collision>
-        <origin xyz="0.0 0.0 0.0" rpy="0.0 1.57075 1.57075"/>
-        <geometry>
-          <cylinder radius="${cyl_rad}" length="0.05"/>
-        </geometry>
-      </collision>
-      <xacro:default_inertial mass="0.5"/>
-    </link>
-    <joint name="l_${body_side}_ankle" type="continuous">
+          <cylinder radius="${cyl_rad - cyl_rad/2}" length="0.05"/>
+        </geometry>
+        <material name="yellow"/>
+      </visual>
+      <collision>
+        <origin xyz="0.0 0.0 0.0" rpy="0.0 1.57075 1.57075"/>
+        <geometry>
+          <cylinder radius="${cyl_rad - cyl_rad/2}" length="0.05"/>
+        </geometry>
+      </collision>
+      <xacro:default_inertial mass="0.5"/>
+    </link>
+    <joint name="l_${body_side}_ankle" type="continuous"> <!--For the movement of the whole track-->
       <axis xyz="0.0 1 0.0"/>
       <origin xyz="0.0 -0.032 0.0" rpy="0.0 0.0 0.0"/>
@@ -586,9 +625,48 @@
       </joint>
     </transmission>
-    <link name="l_${body_side}_track">
+    <!--wheels-->
+    <link name="l_${body_side}_starts_track">
+      <visual name="l_${body_side}_starts_track">
+        <origin xyz="0.0 0.0 0.0" rpy="0.0 1.57075 1.57075"/>
+        <geometry>
+          <cylinder radius="${cyl_rad}" length="0.05"/>
+        </geometry>
+        <material name="yellow"/>
+      </visual>
+      <collision>
+        <origin xyz="0.0 0.0 0.0" rpy="0.0 1.57075 1.57075"/>
+        <geometry>
+          <cylinder radius="${cyl_rad}" length="0.05"/>
+        </geometry>
+      </collision>
+      <xacro:default_inertial mass="0.5"/>
+    </link>
+    <joint name="l_${body_side}_begin_track_joint" type="continuous">
+      <axis xyz="0.0 1 0.0"/>
+      <origin xyz="0.0 0 0.0" rpy="0.0 0.0 0.0"/>
+      <parent link="l_${body_side}_jointed_track"/>
+      <child link="l_${body_side}_starts_track"/>
+    </joint>
+    <transmission name="l_${body_side}_begin_track_joint_trans">
+      <type>transmission_interface/SimpleTransmission</type>
+      <actuator name="${body_side}_l_begin_track_joint_motor">
+        <mechanicalReduction>1</mechanicalReduction>
+      </actuator>
+      <joint name="l_${body_side}_begin_track_joint">
+        <hardwareInterface>hardware_interface/PositionJointInterface</hardwareInterface>
+      </joint>
+    </transmission>
+    <gazebo reference="l_${body_side}_starts_track">
+      <mu1 value="200.0"/>
+      <mu2 value="100.0"/>
+      <kp value="10000000.0" />
+      <kd value="1.0" />
+      <material>Gazebo/Grey</material>
+    </gazebo>
+    <link name="l_${body_side}_track"> <!-- Between the two wheels -->
       <visual name="l_${body_side}_track">
         <origin xyz="0.0 0.0 0.0" rpy="0.0 0.0 0.0"/>
         <geometry>
-          <box size="0.190 0.05 0.06"/>
+          <box size="0.190 0.04 0.06"/>
         </geometry>
         <material name="yellow"/>
@@ -597,5 +675,5 @@
         <origin xyz="0.0 0.0 0.0" rpy="0.0 0.0 0.0"/>
         <geometry>
-          <box size="0.190 0.05 0.06"/>
+          <box size="0.190 0.04 0.06"/>
         </geometry>
       </collision>
@@ -639,5 +717,5 @@
       </joint>
     </transmission>
-    <gazebo reference="r_${body_side}_ends_track">
+    <gazebo reference="l_${body_side}_ends_track">
       <mu1 value="200.0"/>
       <mu2 value="100.0"/>
@@ -656,5 +734,6 @@
   <gazebo>
     <plugin name="gazebo_ros_control" filename="libgazebo_ros_control.so">
-      <robotNamespace>/</robotNamespace>
+      <robotNamespace>/cricket</robotNamespace>
+      <robotSimType>gazebo_ros_control/DefaultRobotHWSim</robotSimType>
     </plugin>
   </gazebo>
